File: hardware/SENSORIC_BOARD/nbiot/sensenet_particlemeter.sch (KiCad schematic (older format))
At the start: 80 parts, among them J1 CONN_01X01, J11 CONN_01X01, J13 BARREL_JACK, J17 CONN_01X01, J18 CONN_01X01, J19 CONN_01X01, J2 CONN_01X01, J20 CONN_01X01, J21 CONN_01X01, J3 CONN_01X01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

Commit message: Zaklad nove verze je hotovy, ted jdu udelat vetsi zmeny v napajeni a layoutu, priprava na shield atd.
Other:
- note removed: "https://www.gme.cz/bipolarni-tranzistor-bcv72-sot23"
- note removed: "nanosim pouzdro"
- moved on the sheet: BT1, C1, C10, C11, C12, C13, C14, C15, C16, C19, C2, C21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

Commit message: Novy rozmer desky, zmena napajeni z LDO na step down, pridany 1000uF na 5V
Parts:
- removed C16: 100uF, Capacitors_SMD:c_elec_5x5.3, symbol CP
- removed U8: LD39050, SNPM:DFN-6-1EP_3x3mm_Pitch0.95mm, symbol LD39050
- added C16: 352pF, SNPM:SMD_0805, symbol C
- added C17: 1000u, SNPM:C_Radial_D10_L16_P5_bottom, symbol CP
- added C18: 470uF, SNPM:C_Radial_D6.3_L11.2_P2.5_bottom, symbol CP
- added D6: 1N5819, Diodes_SMD:SOD-123, symbol D_Schottky
- added D7: LED, SNPM:SMD_0805, symbol LED
- added L5: 41uH, Inductors:Inductor_Taiyo-Yuden_NR-50xx, symbol L
- added L6: 1uH, SNPM:SMD_0805, symbol L
- added R19: 0R33, SNPM:SMD_0805, symbol R
- added R20, R21, R24: tbd, SNPM:SMD_0805, symbol R
- added R22: 18k, SNPM:SMD_0805, symbol R
- added R23: 11k, SNPM:SMD_0805, symbol R
- added R25: 0R1, SNPM:SMD_0805, symbol R
- added R26: 5k6, SNPM:SMD_0805, symbol R
- added U6: MC33063, Housings_SOIC:SOIC-8_3.9x4.9mm_Pitch1.27mm, symbol MC33063
- C12: value 470pF -> 510pF
- C19: footprint Capacitors_ThroughHole:C_Radial_D10_L16_P5 -> SNPM:C_Radial_D10_L16_P5_bottom
- D5: footprint Diodes_ThroughHole:Diode_DO-41_SOD81_Vertical_AnodeUp -> Diodes_SMD:SOD-123
- L3: value 220uH -> 39uH; footprint Inductors_NEOSID:Neosid_Inductor_Sd8 -> Inductors:Inductor_Taiyo-Yuden_NR-50xx
- L4: footprint Inductors_NEOSID:Neosid_Inductor_Sd8 -> SNPM:SMD_0805
- R12: value 0R47 -> 0R33
- R13: value 0R47 -> tbd
- R15: value R -> 27k
- R16: value R -> 9.1k
Connections:
- net labels added: +9V
- wire segments 315 -> 341
- no-connect marks 86 -> 84
Other:
- note added: "VIN 9V, VOUT 3.3V, Iout 500mA, Vripple 5mV, Fmin 50kHz"
- note added: "VIN 9V, VOUT 5V, Iout 500mA, Vripple 5mV, Fmin 50kHz"
- moved on the sheet: C23, C24
