File: hardware/SENSORIC_BOARD/nbiot/sensenet_particlemeter.sch (KiCad schematic (older format))
At the start: 94 parts, among them J1 CONN_01X01, J11 CONN_01X01, J13 BARREL_JACK, J17 CONN_01X01, J18 CONN_01X01, J19 CONN_01X01, J2 CONN_01X01, J20 CONN_01X01, J21 CONN_01X01, J3 CONN_01X01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

Commit message: objednavam prototypy
Parts:
- removed J9: CONN_01X01, SNPM:MountingHole_3.2mm_M3_DIN965, symbol Conn_01x01
- removed P3: CONN_02X11, Pin_Headers:Pin_Header_Straight_2x11, symbol CONN_02X11
- removed SW1: SW_Push, SNPM:SW_DIP_x1_W8.61mm_Slide_SMD_LowProfile, symbol SW_Push
- removed SW2: SW_DIP_x02, Housings_DIP:DIP-4_W7.62mm, symbol SW_DIP_x02
- added D10, D8, D9: LED, SNPM:SMD_0805, symbol LED
- added P3: CONN_02X12, Pin_Headers:Pin_Header_Straight_2x12, symbol CONN_02X12
- added R27, R28, R29: R, SNPM:SMD_0805, symbol R
- added SW1, SW3: SW_DPST, SNPM:edge_switch, symbol SW_DPST
- added SW2: SW_DIP_x03, Housings_DIP:DIP-6_W7.62mm, symbol SW_DIP_x03
Connections:
- net labels added: NETLIGHT, USART_debug_rx, USART_debug_tx, debug_on_off
- wire segments 341 -> 371
- no-connect marks 84 -> 74
Other:
- moved on the sheet: C10, C11, C7, J1, J2, J3, J4, J5, P1, R10, R11, R14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

Commit message: pred debugem noveho hardwaru
Parts:
- removed P4: USB_B, Connectors:USB_Micro-B, symbol USB_B
- added R30: 0R1, SNPM:SMD_0805, symbol R
- added U8: usb_femalee, Connectors:USB_Micro-B, symbol usb_femalee
Connections:
- net +5V: now also R30.1; no longer C15.1, C17.1, C25.1, L4.2
- net GND: now also U8.1 (gnd), U8.6 (shield)
- net PA11-USB-DM: now also U8.4 (D-)
- net PA11-USB-DP renamed PA12-USB-DP
- net PA12-USB-DP: now also U8.3 (D+)
- new net: C15.1, C17.1, C25.1, L4.2, R30.2
- no-connect marks 74 -> 75
Other:
- moved on the sheet: D4, R3
Changed lines of the file:
@@
 L +5V #PWR01
 U 1 1 5995C3C8
-P 22000 1500
-F 0 "#PWR01" H 22000 1350 50  0001 C CNN
-F 1 "+5V" H 22000 1640 50  0000 C CNN
-F 2 "" H 22000 1500 50  0001 C CNN
-F 3 "" H 22000 1500 50  0001 C CNN
-	1    22000 1500
+P 22250 1500
+F 0 "#PWR01" H 22250 1350 50  0001 C CNN
+F 1 "+5V" H 22250 1640 50  0000 C CNN
+F 2 "" H 22250 1500 50  0001 C CNN
+F 3 "" H 22250 1500 50  0001 C CNN
+	1    22250 1500
 	1    0    0    -1
 $EndComp
@@
 L LED D4
 U 1 1 599D2370
-P 21800 2250
-F 0 "D4" H 21800 2350 50  0000 C CNN
-F 1 "LED" H 21800 2150 50  0000 C CNN
-F 2 "SNPM:SMD_0805" H 21800 2250 50  0001 C CNN
-F 3 "" H 21800 2250 50  0001 C CNN
-	1    21800 2250
+P 22050 2250
+F 0 "D4" H 22050 2350 50  0000 C CNN
+F 1 "LED" H 22050 2150 50  0000 C CNN
+F 2 "SNPM:SMD_0805" H 22050 2250 50  0001 C CNN
+F 3 "" H 22050 2250 50  0001 C CNN
+	1    22050 2250
 	0    -1   -1   0
 $EndComp
@@
 L R R3
 U 1 1 599D2485
-P 21800 1750
-F 0 "R3" V 21880 1750 50  0000 C CNN
-F 1 "5k6" V 21800 1750 50  0000 C CNN
-F 2 "SNPM:SMD_0805" V 21730 1750 50  0001 C CNN
-F 3 "" H 21800 1750 50  0001 C CNN
-	1    21800 1750
+P 22050 1750
+F 0 "R3" V 22130 1750 50  0000 C CNN
+F 1 "5k6" V 22050 1750 50  0000 C CNN
+F 2 "SNPM:SMD_0805" V 21980 1750 50  0001 C CNN
+F 3 "" H 22050 1750 50  0001 C CNN
+	1    22050 1750
 	1    0    0    -1
 $EndComp
@@
 L GND #PWR020
 U 1 1 599D2A4C
-P 21800 2550
-F 0 "#PWR020" H 21800 2300 50  0001 C CNN
-F 1 "GND" H 21800 2400 50  0000 C CNN
-F 2 "" H 21800 2550 50  0001 C CNN
-F 3 "" H 21800 2550 50  0001 C CNN
-	1    21800 2550
+P 22050 2550
+F 0 "#PWR020" H 22050 2300 50  0001 C CNN
+F 1 "GND" H 22050 2400 50  0000 C CNN
+F 2 "" H 22050 2550 50  0001 C CNN
+F 3 "" H 22050 2550 50  0001 C CNN
+	1    22050 2550
 	1    0    0    -1
 $EndComp
@@
 $EndComp
 Wire Wire Line
-	20600 1550 22000 1550
+	20600 1550 21650 1550
+Wire Wire Line
+	21950 1550 22250 1550
 Wire Wire Line
 	20850 2150 21500 2150
@@
 	5750 2500 6450 2500
 Wire Wire Line
-	21800 2550 21800 2400
+	22050 2550 22050 2400
 Wire Wire Line
-	21800 2100 21800 1900
+	22050 2100 22050 1900
 Wire Wire Line
-	22000 1550 22000 1500
-Connection ~ 21800 1550
+	22250 1550 22250 1500
+Connection ~ 22050 1550
 Wire Wire Line
 	19650 10300 20100 10300
@@
 Wire Wire Line
 	12950 2500 12950 2600
-$Comp
-L USB_B P4
-U 1 1 5B355601
-P 18050 7200
-F 0 "P4" H 18250 7000 50  0000 C CNN
-F 1 "USB_B" H 18000 7400 50  0000 C CNN
-F 2 "Connectors:USB_Micro-B" V 18000 7100 50  0001 C CNN
-F 3 "" V 18000 7100 50  0000 C CNN
-	1    18050 7200
-	0    1    1    0
-$EndComp
 Text GLabel 6000 2950 2    39   Input ~ 0
 PA11-USB-DM
-Text GLabel 17650 7100 0    39   Input ~ 0
+Text GLabel 17550 8550 0    39   Input ~ 0
 PA11-USB-DM
 Text GLabel 6000 2800 2    39   Input ~ 0
-PA11-USB-DP
-Text GLabel 17650 7200 0    39   Input ~ 0
-PA11-USB-DP
+PA12-USB-DP
+Text GLabel 17550 8400 0    39   Input ~ 0
+PA12-USB-DP
 $Comp
 L GND #PWR061
 U 1 1 5B35767E
-P 17650 7600
-F 0 "#PWR061" H 17650 7350 50  0001 C CNN
-F 1 "GND" H 17650 7450 50  0000 C CNN
-F 2 "" H 17650 7600 50  0001 C CNN
-F 3 "" H 17650 7600 50  0001 C CNN
-	1    17650 7600
+P 17500 8100
+F 0 "#PWR061" H 17500 7850 50  0001 C CNN
+F 1 "GND" H 17500 7950 50  0000 C CNN
+F 2 "" H 17500 8100 50  0001 C CNN
+F 3 "" H 17500 8100 50  0001 C CNN
+	1    17500 8100
 	1    0    0    -1
 $EndComp
-Wire Wire Line
-	17650 7100 17750 7100
-Wire Wire Line
-	17650 7200 17750 7200
-Wire Wire Line
-	17650 7300 17650 7600
-Wire Wire Line
-	17650 7300 17750 7300
-Wire Wire Line
-	17650 7500 18150 7500
-Connection ~ 17650 7500
 Text GLabel 3600 1650 1    39   Input ~ 0
 BOOT_0
@@
 	21500 2150 21500 1950
 Wire Wire Line
-	21500 1650 21500 1550
+	21500 1550 21500 1650
 Connection ~ 21500 1550
 Wire Wire Line
-	21200 1650 21200 1550
+	21200 1550 21200 1650
 $Comp
 L R R12
@@
 	16100 1700 15950 1700
 Wire Wire Line
-	15950 1200 15950 1700
+	15950 1700 15950 1200
 Connection ~ 15950 1200
 Connection ~ 16100 1700
@@
 Wire Wire Line
 	20650 7900 20750 7900
-NoConn ~ 17750 7000
 Wire Notes Line
 	800  1100 800  7600
@@
 $EndComp
 Wire Wire Line
-	21800 1600 21800 1550
+	22050 1600 22050 1550
 Wire Wire Line
 	22300 4500 22300 4450
@@
 Wire Wire Line
 	2300 2500 2500 2500
+$Comp
+L R R30
+U 1 1 5B507155
+P 21800 1550
+F 0 "R30" V 21880 1550 50  0000 C CNN
+F 1 "0R1" V 21800 1550 50  0000 C CNN
+F 2 "SNPM:SMD_0805" V 21730 1550 50  0001 C CNN
+F 3 "" H 21800 1550 50  0001 C CNN
+	1    21800 1550
+	0    1    1    0
+$EndComp
+$Comp
+L usb_femalee U8
+U 1 1 5B54F193
+P 17950 8350
+F 0 "U8" H 17600 8700 60  0000 C CNN
+F 1 "usb_femalee" H 18050 8700 60  0000 C CNN
+F 2 "Connectors:USB_Micro-B" H 17950 8350 60  0001 C CNN
+F 3 "" H 17950 8350 60  0001 C CNN
+	1    17950 8350
+	0    1    1    0
+$EndComp
+NoConn ~ 17750 8250
+NoConn ~ 17750 8700
+Wire Wire Line
+	17500 8100 17750 8100
+Wire Wire Line
+	17500 7750 17500 8100
+Wire Wire Line
+	17500 7750 18200 7750
+Wire Wire Line
+	17550 8400 17750 8400
+Wire Wire Line
+	17550 8550 17750 8550
 $EndSCHEMATC

Commit message: Startovaci bod pro praci na hw 2.0
Other:
- note added: "zamek ke mne, drat doprava, jednicla dole.\n6 gnd\n5 SS\n4 SDI\n3 SDO\n2 SCK\n1 VCC\n"
Changed lines of the file:
@@
 Wire Wire Line
 	17550 8550 17750 8550
+Text Notes 21450 7750 0    60   ~ 0
+zamek ke mne, drat doprava, jednicla dole.\n6 gnd\n5 SS\n4 SDI\n3 SDO\n2 SCK\n1 VCC\n
 $EndSCHEMATC

Commit message: pred displayem
Parts:
- removed BT1: Battery_Cell, SNPM:BAT-CR2032_bottom, symbol Battery_Cell
- removed C1, C2: 4.3p, SNPM:SMD_0805, symbol C
- removed C24: 220n, SNPM:SMD_0805, symbol C
- removed C3: C, SNPM:SMD_0805, symbol C
- removed J17, J20: CONN_01X01, SNPM:Pin_Header_Straight_1x01_Pitch2.54mm, symbol Conn_01x01
- removed L4, L6: 1uH, SNPM:SMD_0805, symbol L
- removed R25, R30: 0R1, SNPM:SMD_0805, symbol R
- removed Y1: 8MHz, Crystals:Crystal_SMD_5032-2pin_5.0x3.2mm, symbol Crystal
- added D11: SM2T3V3A, SNPM:D_SOD-123, symbol D_Schottky
- added L4, L6, L7, L8: FBMH1608HL601-T, Resistors_SMD:R_0603, symbol Ferrite_Bead
- added U9: OLED_128x64, symbol OLED_128x64
- C15: value 1u -> 1000u; footprint SNPM:SMD_0805 -> SNPM:C_Radial_D10_L16_P5_bottom
- D1: value D_Schottky -> PTVS3V3S1UR,115; footprint SNPM:D_SOD-123 -> SNPM:SMD_0805
- D10, D2, D8, D9: footprint SNPM:SMD_0805 -> SNPM:SMD_0805_bottom
- D4: value LED -> red LED; footprint SNPM:SMD_0805 -> SNPM:SMD_0805_bottom
- D5, D6: footprint Diodes_SMD:SOD-123 -> SNPM:D_SOD-123
- D7: value LED -> green LED; footprint SNPM:SMD_0805 -> SNPM:SMD_0805_bottom
- L3, L5: footprint Inductors:Inductor_Taiyo-Yuden_NR-50xx -> SNPM:Inductor_Taiyo-Yuden_NR-50xx
- P1, P2: footprint SNPM:Antenna_conn -> SNPM:Antenna_conn_bot
- P3: footprint Pin_Headers:Pin_Header_Straight_2x12 -> SNPM:Pin_Header_Straight_2x12
- Q1: footprint TO_SOT_Packages_SMD:SOT-23 -> SNPM:SOT-23
- R16: value 9.1k -> 10k
- R22: value 18k -> 8k2
- R23: value 11k -> 5k6
- R26: value 5k6 -> 1k
- R3: value 5k6 -> 8k2
- SW1, SW3: footprint SNPM:edge_switch -> SNPM:edge_switch_bot
- SW2: footprint Housings_DIP:DIP-6_W7.62mm -> SNPM:DIP-6_W7.62mm_bot
- U1: footprint Housings_SOIC:SOIC-8_3.9x4.9mm_Pitch1.27mm -> SNPM:SOIC-8_3.9x4.9mm_Pitch1.27mm
Connections:
- net +3V3: now also C23.1, P3.2 (P2), SW2.5, SW2.6, D11.1 (K), L8.1; no longer P3.3 (P3), SW2.1, SW2.2
- net +5V: now also C15.1, C25.1, D1.1 (K), P3.12 (P12), L7.1; no longer P3.14 (P14)
- net BOOT_0: now also R7.2, SW2.1; no longer R14.2, SW2.5
- net BOOT_signal: now also R14.2, SW2.2; no longer R7.2, SW2.6
- net GND: now also D1.2 (A), P3.22 (P22), SW2.3, D11.2 (A); no longer P3.4 (P4), SW2.4
- net NETLIGHT: now also U2.3 (pc14); no longer U2.2 (pc13)
- net PM_SCK: now also P3.17 (P17); no longer P3.20 (P20)
- net PM_SDI: now also P3.15 (P15); no longer P3.18 (P18)
- net PM_SS: now also P3.18 (P18), U2.54 (pd2); no longer P3.22 (P22), U2.41 (pa8)
- net RI: now also U2.2 (pc13); no longer U2.3 (pc14)
- net Rx: now also P3.19 (P19); no longer P3.13 (P13)
- net SWD_CLK: now also P3.21 (P21); no longer P3.6 (P6)
- net SWD_DIO: now also P3.23 (P23); no longer P3.8 (P8)
- net Tx: now also P3.20 (P20); no longer P3.15 (P15)
- net UART_GPS_RX: now also P3.8 (P8); no longer P3.9 (P9)
- net UART_GPS_TX: now also P3.7 (P7); no longer P3.11 (P11)
- net USART_debug_rx: now also P3.13 (P13); no longer P3.2 (P2)
- net USART_debug_tx: now also P3.14 (P14); no longer P3.1 (P1)
- net WIRELESS_reset: now also P3.10 (P10), U2.53 (pc12); no longer P3.17 (P17), U2.42 (pa9)
- net batt: no longer D1.1 (K), U2.1 (vbat), U7.14 (bv)
- net debug_on_off: now also SW2.4; no longer SW2.3
- net gps_fix: now also P3.9 (P9), U2.15 (pa1); no longer P3.23 (P23), U2.21 (pa5)
- net gps_pulses: now also P3.4 (P4), U2.10 (pc2); no longer P3.19 (P19), U2.24 (pc4)
- net gps_reset: now also P3.5 (P5), U2.11 (pc3); no longer P3.21 (P21), U2.23 (pa7)
- net gps_standby: now also P3.6 (P6), U2.14 (pa0); no longer P3.12 (P12), U2.22 (pa6)
- net i2c_scl: now also P3.3 (P3); no longer P3.7 (P7)
- net i2c_sda: now also P3.1 (P1); no longer P3.5 (P5)
- net reset: now also P3.24 (P24); no longer P3.10 (P10)
- net at C18.1: now also L6.1, L8.2; no longer C23.1
- net at L3.2, R15.1: now also L4.2
- net NMOS: now reaches Q1.3 (D)
- net NMOS: now also P3.11 (P11); no longer P3.24 (P24)
- net at L5.2, R22.1: now also L6.2
- new net: C17.1, L4.1, L7.2
- no-connect marks 75 -> 77
Other:
- note added: "FBMH1608HL601-T"
- note added: "PTVS3V3S1UR,115"
- note added: "SM2T3V3A"
- note added: "VIN 9V, VOUT 3.13V, Iout 500mA, Vripple 5mV, Fmin 50kHz"
- note added: "VIN 9V, VOUT 4,65V, Iout 500mA, Vripple 5mV, Fmin 50kHz"
- note removed: "VIN 9V, VOUT 3.3V, Iout 500mA, Vripple 5mV, Fmin 50kHz"
- note removed: "VIN 9V, VOUT 5V, Iout 500mA, Vripple 5mV, Fmin 50kHz"
- moved on the sheet: C17, C18, C23, D4, J21, L3, Q1, R15, R16, R17, R18, R21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
