File: hardware/SENSORIC_BOARD/nbiot/sensenet_particlemeter.sch (KiCad schematic (older format))
At the start: 102 parts, among them J1 CONN_01X01, J11 CONN_01X01, J13 BARREL_JACK, J18 CONN_01X01, J19 CONN_01X01, J2 CONN_01X01, J21 CONN_01X01, J3 CONN_01X01, J4 CONN_01X01, J5 CONN_01X01, J6 CONN_01X01, P1 SMA_mini, P2 SMA_mini, P3 CONN_02X12, Q1 Q_NMOS_GSD, SW1 SW_DPST, SW2 SW_DIP_x03, SW3 SW_DPST, U1 MC33063, U10 bme280_barebone, U2 stm32f072, U3 QUECTEL_BC95, U4 SIM, U5 CAT24C02, U6 MC33063, U7 M10578-A2, U8 usb_femalee, U9 OLED_128x64

Commit message: snazim se rozchodit novou serii, jebne me z toho z chvili
Parts:
- added C24: 2.2u, SNPM:SMD_0805, symbol C
- added J10, J12, J14, J15, J7, J8, J9: CONN_01X01, SNPM:smd_point_bottom, symbol Conn_01x01
Connections:
- wire segments 392 -> 411
- no-connect marks 87 -> 86
Other:
- note added: "PMEG4010EH,115"
Changed lines of the file:
@@
 	1    0    0    -1
 $EndComp
-NoConn ~ 9750 8800
 NoConn ~ 10050 8800
 NoConn ~ 10150 8800
@@
 	21050 7900 21150 7900
 Wire Wire Line
-	9550 8800 9550 9800
-Wire Wire Line
-	9650 8800 9650 9800
-Wire Wire Line
 	9850 9200 9850 8800
-Wire Wire Line
-	9550 9800 10100 9800
 Wire Wire Line
 	9850 9500 9850 10000
@@
 	1    0    0    -1
 $EndComp
+Wire Wire Line
+	9200 9800 9200 8950
+Wire Wire Line
+	9200 8950 9550 8950
+Wire Wire Line
+	9550 8950 9550 8800
+Wire Wire Line
+	9650 9700 9300 9700
+Wire Wire Line
+	9300 9700 9300 9050
+Wire Wire Line
+	9300 9050 9650 9050
+Wire Wire Line
+	9650 9700 9650 9800
+Wire Wire Line
+	9200 9800 10100 9800
+Wire Wire Line
+	9650 9050 9650 8800
+$Comp
+L C C24
+U 1 1 5BD086E0
+P 9600 9350
+F 0 "C24" H 9625 9450 50  0000 L CNN
+F 1 "2.2u" H 9625 9250 50  0000 L CNN
+F 2 "SNPM:SMD_0805" H 9638 9200 50  0001 C CNN
+F 3 "" H 9600 9350 50  0001 C CNN
+	1    9600 9350
+	1    0    0    -1
+$EndComp
+Wire Wire Line
+	9600 9200 9600 9150
+Wire Wire Line
+	9600 9150 9750 9150
+Wire Wire Line
+	9750 9150 9750 8800
+Wire Wire Line
+	9600 9500 9600 9600
+Wire Wire Line
+	9600 9600 9750 9600
+Wire Wire Line
+	9750 9600 9750 9800
+Connection ~ 9750 9800
+$Comp
+L Conn_01x01 J7
+U 1 1 5BD0A84C
+P 9700 10800
+F 0 "J7" V 9700 10700 50  0000 C CNN
+F 1 "CONN_01X01" V 9800 10800 50  0001 C CNN
+F 2 "SNPM:smd_point_bottom" H 9700 10800 50  0001 C CNN
+F 3 "" H 9700 10800 50  0001 C CNN
+	1    9700 10800
+	0    -1   -1   0
+$EndComp
+$Comp
+L Conn_01x01 J8
+U 1 1 5BD0BD5A
+P 9950 10800
+F 0 "J8" V 9950 10700 50  0000 C CNN
+F 1 "CONN_01X01" V 10050 10800 50  0001 C CNN
+F 2 "SNPM:smd_point_bottom" H 9950 10800 50  0001 C CNN
+F 3 "" H 9950 10800 50  0001 C CNN
+	1    9950 10800
+	0    -1   -1   0
+$EndComp
+$Comp
+L Conn_01x01 J9
+U 1 1 5BD0BEAB
+P 10200 10800
+F 0 "J9" V 10200 10700 50  0000 C CNN
+F 1 "CONN_01X01" V 10300 10800 50  0001 C CNN
+F 2 "SNPM:smd_point_bottom" H 10200 10800 50  0001 C CNN
+F 3 "" H 10200 10800 50  0001 C CNN
+	1    10200 10800
+	0    -1   -1   0
+$EndComp
+$Comp
+L Conn_01x01 J10
+U 1 1 5BD0BFFF
+P 10450 10800
+F 0 "J10" V 10450 10700 50  0000 C CNN
+F 1 "CONN_01X01" V 10550 10800 50  0001 C CNN
+F 2 "SNPM:smd_point_bottom" H 10450 10800 50  0001 C CNN
+F 3 "" H 10450 10800 50  0001 C CNN
+	1    10450 10800
+	0    -1   -1   0
+$EndComp
+$Comp
+L Conn_01x01 J12
+U 1 1 5BD0C156
+P 10700 10800
+F 0 "J12" V 10700 10700 50  0000 C CNN
+F 1 "CONN_01X01" V 10800 10800 50  0001 C CNN
+F 2 "SNPM:smd_point_bottom" H 10700 10800 50  0001 C CNN
+F 3 "" H 10700 10800 50  0001 C CNN
+	1    10700 10800
+	0    -1   -1   0
+$EndComp
+$Comp
+L Conn_01x01 J14
+U 1 1 5BD0C2BC
+P 10950 10800
+F 0 "J14" V 10950 10700 50  0000 C CNN
+F 1 "CONN_01X01" V 11050 10800 50  0001 C CNN
+F 2 "SNPM:smd_point_bottom" H 10950 10800 50  0001 C CNN
+F 3 "" H 10950 10800 50  0001 C CNN
+	1    10950 10800
+	0    -1   -1   0
+$EndComp
+$Comp
+L Conn_01x01 J15
+U 1 1 5BD0C419
+P 11200 10800
+F 0 "J15" V 11200 10700 50  0000 C CNN
+F 1 "CONN_01X01" V 11300 10800 50  0001 C CNN
+F 2 "SNPM:smd_point_bottom" H 11200 10800 50  0001 C CNN
+F 3 "" H 11200 10800 50  0001 C CNN
+	1    11200 10800
+	0    -1   -1   0
+$EndComp
+$Comp
+L GND #PWR093
+U 1 1 5BD0C6C7
+P 11200 11150
+F 0 "#PWR093" H 11200 10900 50  0001 C CNN
+F 1 "GND" H 11200 11000 50  0000 C CNN
+F 2 "" H 11200 11150 50  0001 C CNN
+F 3 "" H 11200 11150 50  0001 C CNN
+	1    11200 11150
+	1    0    0    -1
+$EndComp
+$Comp
+L +5V #PWR094
+U 1 1 5BD0D1A9
+P 10950 11150
+F 0 "#PWR094" H 10950 11000 50  0001 C CNN
+F 1 "+5V" H 10950 11290 50  0000 C CNN
+F 2 "" H 10950 11150 50  0001 C CNN
+F 3 "" H 10950 11150 50  0001 C CNN
+	1    10950 11150
+	-1   0    0    1
+$EndComp
+Text GLabel 10700 11150 3    39   Input ~ 0
+PM_SCK
+Text GLabel 10450 11150 3    39   Input ~ 0
+PM_SDO
+Text GLabel 10200 11150 3    39   Input ~ 0
+OLED_RESET
+Text GLabel 9950 11150 3    39   Input ~ 0
+OLED_D/C
+Text GLabel 9700 11150 3    39   Input ~ 0
+OLED_CS
+Wire Wire Line
+	9700 11000 9700 11150
+Wire Wire Line
+	9950 11000 9950 11150
+Wire Wire Line
+	10200 11000 10200 11150
+Wire Wire Line
+	10450 11000 10450 11150
+Wire Wire Line
+	10700 11000 10700 11150
+Wire Wire Line
+	10950 11000 10950 11150
+Wire Wire Line
+	11200 11000 11200 11150
+Text Notes 14800 1000 0    60   ~ 0
+PMEG4010EH,115
 $EndSCHEMATC

Commit message: zonglovani s repama
Parts:
- C1, C10, C11, C13, C14, C15, C16, C2, C20, C21, C22, C23, C24, C25, C3, C4, C5, C6, C7, C8, C9: symbol C -> sensenet_particlemeter-rescue:C
- C12: value 510pF -> 330pF; symbol C -> sensenet_particlemeter-rescue:C
- C17, C18, C19: symbol CP -> sensenet_particlemeter-rescue:CP
- D1, D11, D3, D5, D6: symbol D_Schottky -> sensenet_particlemeter-rescue:D_Schottky
- D10, D2, D4, D7, D8, D9: symbol LED -> sensenet_particlemeter-rescue:LED
- J1, J10, J11, J12, J14, J15, J18, J19, J2, J21, J3, J4, J5, J6, J7, J8, J9: symbol Conn_01x01 -> sensenet_particlemeter-rescue:Conn_01x01
- J13: symbol Barrel_Jack -> sensenet_particlemeter-rescue:Barrel_Jack
- L1, L2, L3, L5: symbol L -> sensenet_particlemeter-rescue:L
- L4, L6, L7, L8: symbol Ferrite_Bead -> sensenet_particlemeter-rescue:Ferrite_Bead
- LOGO1: symbol LOGO -> sensenet_particlemeter-rescue:LOGO
- P1, P2: symbol SMA_mini -> sensenet_particlemeter-rescue:SMA_mini
- P3: symbol CONN_02X12 -> sensenet_particlemeter-rescue:CONN_02X12
- Q1: symbol Q_NMOS_GSD -> sensenet_particlemeter-rescue:Q_NMOS_GSD
- R1, R10, R11, R12, R13, R14, R17, R18, R19, R2, R20, R22, R23, R24, R25, R26, R27, R28, R29, R3, R4, R5, R6, R7, R8, R9: symbol R -> sensenet_particlemeter-rescue:R
- R15: value 27k -> 2k7; symbol R -> sensenet_particlemeter-rescue:R
- R16: value 10k -> 820R; symbol R -> sensenet_particlemeter-rescue:R
- R21: value tbd -> 100R; symbol R -> sensenet_particlemeter-rescue:R
- SJ16: symbol solder_jumper -> sensenet_particlemeter-rescue:solder_jumper
- SW1, SW3: symbol SW_DPST -> sensenet_particlemeter-rescue:SW_DPST
- SW2: symbol SW_DIP_x03 -> sensenet_particlemeter-rescue:SW_DIP_x03
- U1, U6: symbol MC33063 -> sensenet_particlemeter-rescue:MC33063
- U10: symbol bme280_barebone -> sensenet_particlemeter-rescue:bme280_barebone
- U2: symbol stm32f072 -> sensenet_particlemeter-rescue:stm32f072
- U3: symbol QUECTEL_BC95 -> sensenet_particlemeter-rescue:QUECTEL_BC95
- U4: symbol SIM -> sensenet_particlemeter-rescue:SIM
- U5: symbol CAT24C02 -> sensenet_particlemeter-rescue:CAT24C02
- U7: symbol M10578-A2 -> sensenet_particlemeter-rescue:M10578-A2
- U8: symbol usb_femalee -> sensenet_particlemeter-rescue:usb_femalee
- U9: symbol OLED_128x64 -> sensenet_particlemeter-rescue:OLED_128x64
Connections:
- wire segments 411 -> 498

Commit message: rozdelane upravicky
Parts:
- removed C17: 1000u, SNPM:C_Radial_D10_L16_P5_bottom, symbol sensenet_particlemeter-rescue:CP
- removed J13: BARREL_JACK, SNPM:BARREL_JACK, symbol sensenet_particlemeter-rescue:Barrel_Jack
- added C17: 100n, Capacitor_SMD:C_0805_2012Metric, symbol sensenet_particlemeter-rescue:C
- added C26, C27: 1n, Capacitor_SMD:C_0805_2012Metric, symbol sensenet_particlemeter-rescue:C
- added C28: 22p, Capacitor_SMD:C_0805_2012Metric, symbol sensenet_particlemeter-rescue:C
- added J13: Conn_01x02_Female, Connector_Wire:SolderWirePad_1x02_P3.81mm_Drill1.2mm, symbol Connector:Conn_01x02_Female
- added L9: 39uH, Inductor_SMD:L_Taiyo-Yuden_NR-50xx, symbol sensenet_particlemeter-rescue:L
- added R30: 0R, Resistor_SMD:R_0805_2012Metric, symbol Device:R
- C13: value C -> 100n
- C15: value 1000u -> 470u; footprint SNPM:C_Radial_D10_L16_P5_bottom -> Capacitor_SMD:C_0805_2012Metric
- C18: footprint SNPM:C_Radial_D6.3_L11.2_P2.5_bottom -> Capacitor_THT:CP_Radial_D10.0mm_P5.00mm
- C19: footprint SNPM:C_Radial_D10_L16_P5_bottom -> Capacitor_THT:CP_Radial_D10.0mm_P5.00mm
- L1, L2: value L -> DNP
Connections:
- net labels added: 5V_enable
- net labels removed: batt
- wire segments 498 -> 513
- no-connect marks 86 -> 85
Other:
- moved on the sheet: C15, C19, C25, C7, D1, D3, L4, L7, R12, R13, U4

Commit message: V5
Parts:
- removed D4: red LED, SNPM:SMD_0805_bottom, symbol sensenet_particlemeter-rescue:LED
- removed D5: 1N5819, SNPM:D_SOD-123, symbol sensenet_particlemeter-rescue:D_Schottky
- removed D7: green LED, SNPM:SMD_0805_bottom, symbol sensenet_particlemeter-rescue:LED
- removed L9: 39uH, Inductor_SMD:L_Taiyo-Yuden_NR-50xx, symbol sensenet_particlemeter-rescue:L
- removed R15: 2k7, SNPM:SMD_0805, symbol sensenet_particlemeter-rescue:R
- removed R24: tbd, SNPM:SMD_0805, symbol sensenet_particlemeter-rescue:R
- removed R26: 1k, SNPM:SMD_0805, symbol sensenet_particlemeter-rescue:R
- removed R3: 8k2, SNPM:SMD_0805, symbol sensenet_particlemeter-rescue:R
- removed U1: MC33063, SNPM:SOIC-8_3.9x4.9mm_Pitch1.27mm, symbol sensenet_particlemeter-rescue:MC33063
- added C29: 1n, Capacitor_SMD:C_0805_2012Metric, symbol sensenet_particlemeter-rescue:C
- added C30: 47u, Capacitor_SMD:C_0805_2012Metric, symbol sensenet_particlemeter-rescue:C
- added U1: NCP59152, Package_DFN_QFN:DFN-8-1EP_4x4mm_P0.8mm_EP2.39x2.21mm, symbol NCP59152:NCP59152
- C12: value 330pF -> 100n
- C13: value 100n -> 1u
- C15: footprint Capacitor_SMD:C_0805_2012Metric -> Capacitor_THT:CP_Radial_D10.0mm_P5.00mm
- C19: value 1000u -> 470u
- C25: footprint SNPM:SMD_0805 -> Capacitor_SMD:C_0805_2012Metric
- D1: footprint SNPM:SMD_0805 -> Diode_SMD:D_SOD-123
- R12: value 0R33 -> 100k
- R13: value tbd -> 100k
Connections:
- net +9V: now also C12.1, L3.2, C29.1, U1.3 (VIN); no longer R12.2, R13.2
- net 5V_enable: now also R13.1, U1.2 (EN)
- net GND: now also R13.2, R23.2, C29.2, C30.2, U1.1 (GND), U1.9 (heatsink_GND)
- net at D3.1 (K): now also L3.1
- net at R12.1: now also L4.2, R16.1, C30.1, U1.6 (VOUT); no longer R13.1
- net at R16.2, R21.1: now also U1.7 (ADJ)
- new net: R12.2, U1.8 (FLG)
Other:
- note added: "ESE477M025AH1EA"
- note removed: "VIN 9V, VOUT 4,65V, Iout 500mA, Vripple 5mV, Fmin 50kHz"
- moved on the sheet: C13, C19, D3, J13, L3, R16, R21

Commit message: dalsi updaty
Parts:
- removed C20, C22, C3: C, SNPM:SMD_0805, symbol sensenet_particlemeter-rescue:C
- removed C24: 2.2u, SNPM:SMD_0805, symbol sensenet_particlemeter-rescue:C
- removed R25: R, SNPM:SMD_0805, symbol sensenet_particlemeter-rescue:R
- removed U9: OLED_128x64, SNPM:OLED_display128x64_bottom, symbol sensenet_particlemeter-rescue:OLED_128x64
- C1: value 2.2u -> 100n; footprint SNPM:SMD_0805 -> Capacitor_SMD:C_0805_2012Metric
- C10, C11, C12, C13, C14, C16, C4, C5, C6, C7, C8, C9: footprint SNPM:SMD_0805 -> Capacitor_SMD:C_0805_2012Metric
- C2: value C -> 22p; footprint SNPM:SMD_0805 -> Capacitor_SMD:C_0805_2012Metric
- C23: value 10u -> 2.2u
- R16: value 820R -> 3k3
- R21: value 100R -> 1k1
Connections:
- net +3V3: now also C1.1
- no-connect marks 85 -> 75
Other:
- note added: "pico clasp konektor,\n"
- moved on the sheet: C23, D11

Commit message: Daily update, rework zdroju - oba dva LDO s adjustem, 5Venable, pico clasp connector, priprava na lorawan shield
Parts:
- removed C21: 100n, SNPM:SMD_0805, symbol sensenet_particlemeter-rescue:C
- removed D6: 1N5819, SNPM:D_SOD-123, symbol sensenet_particlemeter-rescue:D_Schottky
- removed J10, J12, J14, J15, J7, J8, J9: CONN_01X01, SNPM:smd_point_bottom, symbol sensenet_particlemeter-rescue:Conn_01x01
- removed P3: CONN_02X12, SNPM:Pin_Header_Straight_2x12, symbol sensenet_particlemeter-rescue:CONN_02X12
- removed Q1: Q_NMOS_GSD, SNPM:SOT-23, symbol sensenet_particlemeter-rescue:Q_NMOS_GSD
- removed R14, R7: 10k, SNPM:SMD_0805, symbol sensenet_particlemeter-rescue:R
- removed R17, R18: R, SNPM:SMD_0805, symbol sensenet_particlemeter-rescue:R
- removed R19: 0R33, SNPM:SMD_0805, symbol sensenet_particlemeter-rescue:R
- removed R2, R5: 4.7k, SNPM:SMD_0805, symbol sensenet_particlemeter-rescue:R
- removed R6: 22k, SNPM:SMD_0805, symbol sensenet_particlemeter-rescue:R
- removed SJ16: solder_jumper, SNPM:solder_jumper, symbol sensenet_particlemeter-rescue:solder_jumper
- removed SW2: SW_DIP_x03, SNPM:DIP-6_W7.62mm_bot, symbol sensenet_particlemeter-rescue:SW_DIP_x03
- removed U10: bme280_barebone, SNPM:BME280, symbol sensenet_particlemeter-rescue:bme280_barebone
- removed U5: CAT24C02, TO_SOT_Packages_SMD:SOT-23-5, symbol sensenet_particlemeter-rescue:CAT24C02
- removed U6: MC33063, Housings_SOIC:SOIC-8_3.9x4.9mm_Pitch1.27mm, symbol sensenet_particlemeter-rescue:MC33063
- removed U8: usb_femalee, Connectors:USB_Micro-B, symbol sensenet_particlemeter-rescue:usb_femalee
- added C20: 100n, Capacitor_SMD:C_0805_2012Metric, symbol sensenet_particlemeter-rescue:C
- added C22, C24: 1n, Capacitor_SMD:C_0805_2012Metric, symbol sensenet_particlemeter-rescue:C
- added C3: 22u, Capacitor_SMD:C_0805_2012Metric, symbol sensenet_particlemeter-rescue:C
- added J16: Conn_01x06_Female, molexpico:pico_clasp_6_horizontal, symbol Connector:Conn_01x06_Female
- added J17: Conn_02x08_Odd_Even, Connector_PinSocket_2.54mm:PinSocket_2x08_P2.54mm_Vertical, symbol Connector_Generic:Conn_02x08_Odd_Even
- added J20: Conn_02x04_Odd_Even, Connector_PinSocket_2.54mm:PinSocket_2x04_P2.54mm_Vertical, symbol Connector_Generic:Conn_02x04_Odd_Even
- added J7: Conn_01x07_Female, Connector_PinHeader_2.54mm:PinHeader_1x07_P2.54mm_Vertical, symbol Connector:Conn_01x07_Female
- added J8: Conn_01x02_Female, Connector_PinSocket_2.54mm:PinSocket_1x02_P2.54mm_Vertical, symbol Connector:Conn_01x02_Female
- added R3: 4k7, Resistor_SMD:R_0805_2012Metric, symbol sensenet_particlemeter-rescue:R
- added U6: NCP59152, Package_DFN_QFN:DFN-8-1EP_4x4mm_P0.8mm_EP2.39x2.21mm, symbol NCP59152:NCP59152
- added U8: ATECC508A, Package_DFN_QFN:DFN-8-1EP_3x2mm_P0.5mm_EP1.75x1.45mm, symbol atec508A:ATECC508A
- C13: value 1u -> 22u
- C16: value 352pF -> 47u
- C23: value 2.2u -> 100n
- R1, R10, R11, R12, R13, R16, R21, R22, R23, R27, R28, R29, R8, R9: footprint SNPM:SMD_0805 -> Resistor_SMD:R_0805_2012Metric
- R20: value tbd -> 100k; footprint SNPM:SMD_0805 -> Resistor_SMD:R_0805_2012Metric
- R4: value 4.7k -> 4k7; footprint SNPM:SMD_0805 -> Resistor_SMD:R_0805_2012Metric
Connections:
- net +3V3: now also C18.1, R4.1, J20.7 (Pin_7), R3.1, U8.8 (VCC); no longer C23.1, R4.2
- net +5V: now also J16.6 (Pin_6), J17.15 (Pin_15), J17.16 (Pin_16), J7.6 (Pin_6)
- net 5V_enable: now also U2.25 (pc5); no longer U2.26 (pb0)
- net GND: now also C20.2, C22.2, C24.2, C3.2, J16.1 (Pin_1), J17.1 (Pin_1), J17.11 (Pin_11), J17.12 (Pin_12), J17.2 (Pin_2), J17.3 (Pin_3), J20.3 (Pin_3), J20.6 (Pin_6), J20.8 (Pin_8), J7.7 (Pin_7), U6.1 (GND), U6.9 (heatsink_GND), U8.4 (GND)
- net OLED_CS: now also J7.1 (Pin_1)
- net OLED_D/C: now also J7.2 (Pin_2)
- net OLED_RESET: now also J7.3 (Pin_3)
- net PM_SCK: now also J16.5 (Pin_5), J7.5 (Pin_5)
- net PM_SDI: now also J16.3 (Pin_3)
- net PM_SDO: now also J16.4 (Pin_4), J7.4 (Pin_4)
- net PM_SS: now also J16.2 (Pin_2)
- net Rx: now also J20.2 (Pin_2)
- net SWD_CLK: now also J20.5 (Pin_5)
- net SWD_DIO: now also J20.1 (Pin_1)
- net Tx: now also J20.4 (Pin_4)
- net UART_GPS_RX: now also J17.8 (Pin_8)
- net UART_GPS_TX: now also J17.7 (Pin_7)
- net USART_debug_rx: now also J17.14 (Pin_14)
- net USART_debug_tx: now also J17.13 (Pin_13)
- net WIRELESS_reset: now also J17.10 (Pin_10)
- net gps_fix: now also J17.9 (Pin_9)
- net gps_pulses: now also J17.4 (Pin_4)
- net gps_reset: now also J17.5 (Pin_5)
- net gps_standby: now also J17.6 (Pin_6)
- net i2c_scl: now also J8.2 (Pin_2), R3.2, U8.6 (SCL)
- net i2c_sda: now also R4.2, J8.1 (Pin_1), U8.5 (SDA); no longer R4.1
- net at R27.1: now also U2.26 (pb0); no longer U2.25 (pc5)
- net at R20.1: now also U6.8 (FLG)
- net at L6.2, R22.1: now also C16.1, R20.2, U6.6 (VOUT); no longer L5.2
- net +6V: now reaches L5.1
- net +6V: now also C12.1, C13.1, C19.1, C29.1, L3.2, U1.3 (VIN)
- net at L6.1, L8.2: now also C23.1, C24.1; no longer C18.1
- removed net +9V: C12.1, C13.1, C19.1, C29.1, L3.2, R20.2, U1.3 (VIN)
- net PA11-USB-DM: no longer names the net of U2.44 (pa11)
- net PA12-USB-DP: no longer names the net of U2.45 (pa12)
- net PM_meter_switch: no longer names the net of U2.43 (pa10)
- new net: C20.1, C22.1, C3.1, L5.2, U6.3 (VIN)
- no-connect marks 75 -> 80
Other:
- note added: "15133-0601"
- note added: "501568-0607"
- note removed: "VIN 9V, VOUT 3.13V, Iout 500mA, Vripple 5mV, Fmin 50kHz"
- note removed: "po startupu se nacte hodnota \nbootsignal, pokud bude prepinac \nv poloze/usbdfu, tak se nastartuje \nv optionbytech procak jako usbdfu."
- moved on the sheet: C16, C18, C23, D8, L5, L6, R20, R22, R23, R27
