File: hardware/SENSORIC_BOARD/nbiot/_saved_sensenet_particlemeter.sch (KiCad schematic (older format))
At the start: 102 parts, among them J1 CONN_01X01, J11 CONN_01X01, J13 BARREL_JACK, J18 CONN_01X01, J19 CONN_01X01, J2 CONN_01X01, J21 CONN_01X01, J3 CONN_01X01, J4 CONN_01X01, J5 CONN_01X01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

Commit message: novy hw
Parts:
- C2, C20, C22: value C -> 1u
- C3: value C -> 100n
- R25: value R -> 390k
