File: hardware/SENSORIC_BOARD/lorawan/sensenet_particlemeter.kicad_pcb (KiCad board)
At the start: 2 copper layers, 63.6 x 72.3 mm, 89 parts, among them J1 CONN_01X01, J11 CONN_01X01, J13 BARREL_JACK, J17 CONN_01X01, J18 CONN_01X01, J19 CONN_01X01, J20 CONN_01X01, J3 CONN_01X01, J4 CONN_01X01, J5 CONN_01X01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

Commit message: objednavam prototypy
Parts:
- removed J9: CONN_01X01, SNPM:MountingHole_3.2mm_M3_DIN965
- added D10: LED, SNPM:SMD_0805, F.Cu at (172.3, 122.8)
- added D8: LED, SNPM:SMD_0805, F.Cu at (166.2, 122.8)
- added D9: LED, SNPM:SMD_0805, F.Cu at (169.2, 122.8)
- added R27: R, SNPM:SMD_0805, F.Cu at (171.7, 115.7)
- added R28: R, SNPM:SMD_0805, F.Cu at (173.9, 115.7)
- added R29: R, SNPM:SMD_0805, F.Cu at (176.1, 115.7)
- added SW3: SW_DPST, SNPM:edge_switch, F.Cu at (179.1, 123.8)
- P3: value CONN_02X11 -> CONN_02X12; footprint Pin_Headers:Pin_Header_Straight_2x11 -> Pin_Headers:Pin_Header_Straight_2x12
- SW1: value SW_Push -> SW_DPST; footprint SNPM:SW_DIP_x1_W8.61mm_Slide_SMD_LowProfile -> SNPM:edge_switch
- SW2: value SW_DIP_x02 -> SW_DIP_x03; footprint Housings_DIP:DIP-4_W7.62mm -> Housings_DIP:DIP-6_W7.62mm
- moved R3 23.9 mm to (145.6, 115.4)
- moved R26 21.3 mm to (150.6, 115.4)
- moved D7 20.0 mm to (152.1, 123.9)
- moved D4 19.9 mm to (148.1, 123.9), turned to 180 degrees
- moved SW1 11.5 mm to (176.3, 55.1)
- moved SW2 11.4 mm to (172.8, 65.3)
- moved J1 7.62 mm to (144.8, 96.5)
- moved D3 6.54 mm to (181.5, 115.9), turned to 270 degrees
- moved R7 6.01 mm to (181.1, 78.5)
- moved R14 5.88 mm to (181.1, 76.5)
- moved C19 3.77 mm to (180.8, 119.4), turned to 180 degrees
- moved C20 2.75 mm to (133.7, 74.5)
- moved C7 2.64 mm to (157.7, 79.5)
- moved P3 2.55 mm to (191.5, 61.8)
- moved R4 2.53 mm to (193.2, 58.0), turned to 90 degrees
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Connections:
- J1 pad 1: WIRELESS_reset -> Net-(J1-Pad1)
- J4 pad 1: Net-(J4-Pad1) -> WIRELESS_reset
- P3 pad 1: +3V3 -> USART_debug_tx
- P3 pad 10: gps_standby -> reset
- P3 pad 11: Rx -> UART_GPS_TX
- P3 pad 12: +5V -> gps_standby
- P3 pad 13: Tx -> Rx
- P3 pad 14: PM_SDO -> +5V
- P3 pad 15: WIRELESS_reset -> Tx
- P3 pad 16: PM_SDI -> PM_SDO
- P3 pad 17: gps_pulses -> WIRELESS_reset
- P3 pad 18: PM_SCK -> PM_SDI
- P3 pad 19: gps_reset -> gps_pulses
- P3 pad 2: GND -> USART_debug_rx
- P3 pad 20: PM_SS -> PM_SCK
- P3 pad 21: gps_fix -> gps_reset
- P3 pad 22: Net-(P3-Pad22) -> PM_SS
- P3 pad 3: i2c_sda -> +3V3
- P3 pad 4: SWD_CLK -> GND
- P3 pad 5: i2c_scl -> i2c_sda
- P3 pad 6: SWD_DIO -> SWD_CLK
- P3 pad 7: UART_GPS_RX -> i2c_scl
- P3 pad 8: reset -> SWD_DIO
- P3 pad 9: UART_GPS_TX -> UART_GPS_RX
- Q1 pad 3: Net-(P3-Pad22) -> Net-(P3-Pad24)
- SW2 pad 3: BOOT_0 -> debug_on_off
- SW2 pad 4: BOOT_signal -> GND
- U2 pad 25: (no net) -> Net-(R27-Pad1)
- U2 pad 27: (no net) -> Net-(R28-Pad1)
- U2 pad 28: (no net) -> Net-(R29-Pad1)
- U2 pad 29: (no net) -> Net-(SW3-Pad1)
- U2 pad 58: (no net) -> USART_debug_tx
- U2 pad 59: (no net) -> USART_debug_rx
- U2 pad 62: (no net) -> debug_on_off
- U3 pad 30: Net-(J3-Pad1) -> Net-(J1-Pad1)
- U3 pad 31: Net-(J4-Pad1) -> Net-(J3-Pad1)
Routing:
- net +5V: track 38.5 -> 167.3 mm, vias 1 -> 2
- net Net-(SW3-Pad1): track 0.00 -> 38.9 mm
- net USART_debug_rx: track 0.00 -> 32.5 mm
- net Net-(R29-Pad1): track 0.00 -> 32.0 mm
- net Net-(J1-Pad1): track 0.00 -> 31.4 mm
- net GND: track 180.9 -> 150.2 mm, vias 33 -> 25
- net Net-(R28-Pad1): track 0.00 -> 30.4 mm
- net Net-(R27-Pad1): track 0.00 -> 30.0 mm
- net Net-(J4-Pad1): track 28.6 -> 0.00 mm
- net USART_debug_tx: track 0.00 -> 26.1 mm
- net +3V3: track 234.8 -> 254.2 mm, vias 12 -> 14
- net debug_on_off: track 0.00 -> 16.0 mm
- net i2c_scl: track 58.4 -> 70.7 mm, vias 3 -> 5
- net reset: track 46.2 -> 56.7 mm, vias 2 -> 4
- net BOOT_0: track 8.83 -> 18.2 mm
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Other:
- net class Default: trace_width 0.15 -> 0.5
