File: hardware/SENSORIC_BOARD/lorawan/sensenet_particlemeter.sch (KiCad schematic (older format))
At the start: 94 parts, among them J1 CONN_01X01, J11 CONN_01X01, J13 BARREL_JACK, J17 CONN_01X01, J18 CONN_01X01, J19 CONN_01X01, J2 CONN_01X01, J20 CONN_01X01, J21 CONN_01X01, J3 CONN_01X01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

Commit message: zonglovani zase s gitem
Parts:
- removed J2, J21: CONN_01X01, SNPM:Pin_Header_Straight_1x01_Pitch1.00mm, symbol Conn_01x01
- removed R10: 10k, SNPM:SMD_0805, symbol R
- removed R8, R9: 1k, SNPM:SMD_0805, symbol R
- removed U3: QUECTEL_BC95, SNPM:quectel_BC95, symbol QUECTEL_BC95
- removed U4: SIM, SNPM:nanosimmm, symbol SIM
- added C20: 100n, SNPM:SMD_0805, symbol C
- added U3: RN2483, lorawan_module:RN2483_top, symbol RN2483
Connections:
- net labels removed: RI
- wire segments 341 -> 302
- no-connect marks 84 -> 57
Other:
- moved on the sheet: C10, C11, C7, J1, J3, J4, P1, R11

Commit message: objednavam prototypy
Parts:
- removed J9: CONN_01X01, SNPM:MountingHole_3.2mm_M3_DIN965, symbol Conn_01x01
- removed P3: CONN_02X11, Pin_Headers:Pin_Header_Straight_2x11, symbol CONN_02X11
- removed SW1: SW_Push, SNPM:SW_DIP_x1_W8.61mm_Slide_SMD_LowProfile, symbol SW_Push
- removed SW2: SW_DIP_x02, Housings_DIP:DIP-4_W7.62mm, symbol SW_DIP_x02
- added D10, D8, D9: LED, SNPM:SMD_0805, symbol LED
- added P3: CONN_02X12, Pin_Headers:Pin_Header_Straight_2x12, symbol CONN_02X12
- added R27, R28, R29: R, SNPM:SMD_0805, symbol R
- added SW1, SW3: SW_DPST, SNPM:edge_switch, symbol SW_DPST
- added SW2: SW_DIP_x03, Housings_DIP:DIP-6_W7.62mm, symbol SW_DIP_x03
Connections:
- net +3V3: now also P3.3 (P3), SW2.1, SW2.2
- net +5V: now also P3.14 (P14)
- net BOOT_0: now also SW2.5
- net BOOT_signal: now also SW2.6
- net GND: now also D10.1 (K), D8.1 (K), D9.1 (K), P3.4 (P4), SW1.1, SW1.3, SW1.4, SW2.4, SW3.2, SW3.3, SW3.4
- net PM_SCK: now also P3.20 (P20)
- net PM_SDI: now also P3.18 (P18)
- net PM_SDO: now also P3.16 (P16)
- net PM_SS: now also P3.22 (P22)
- net Rx: now also P3.13 (P13)
- net SWD_CLK: now also P3.6 (P6)
- net SWD_DIO: now also P3.8 (P8)
- net Tx: now also P3.15 (P15)
- net UART_GPS_RX: now also P3.9 (P9)
- net UART_GPS_TX: now also P3.11 (P11)
- net WIRELESS_reset: now also J4.1 (Pin_1), P3.17 (P17); no longer J1.1 (Pin_1)
- net gps_fix: now also P3.23 (P23)
- net gps_pulses: now also P3.19 (P19)
- net gps_reset: now also P3.21 (P21)
- net gps_standby: now also P3.12 (P12)
- net i2c_scl: now also P3.7 (P7)
- net i2c_sda: now also P3.5 (P5)
- net reset: now also P3.10 (P10), SW1.2
- net NETLIGHT: now reaches U2.2 (pc13)
- net at U2.25 (pc5): now also R27.1
- net at U2.27 (pb1): now also R28.1
- net at U2.28 (pb2): now also R29.1
- net at U2.29 (pb10): now also SW3.1
- net RI: now reaches U2.3 (pc14)
- net USART_debug_tx: now reaches U2.58 (pb6)
- net USART_debug_tx: now also P3.1 (P1)
- net USART_debug_rx: now reaches U2.59 (pb7)
- net USART_debug_rx: now also P3.2 (P2)
- net debug_on_off: now reaches U2.62 (pb9)
- net debug_on_off: now also SW2.3
- net at J3.1 (Pin_1): now also U3.31 (TEST1); no longer U3.30 (TEST0)
- net at Q1.3 (D): now also P3.24 (P24)
- new net: J1.1 (Pin_1), U3.30 (TEST0)
- new net: D8.2 (A), R27.2
- new net: D9.2 (A), R28.2
- new net: D10.2 (A), R29.2
- no-connect marks 57 -> 47
Other:
- moved on the sheet: C10, C11, C7, J1, J3, J4, J5, P1, R11, R14
