File: hardware/NBIOT_mainboard/sensenet_particlemeter.kicad_pcb (KiCad board)
At the start: 2 copper layers, 63.6 x 72.4 mm, 97 parts, among them J1 CONN_01X01, J11 CONN_01X01, J13 Conn_01x02_Female, J16 Conn_01x06_Female, J17 Conn_02x08_Odd_Even, J18 CONN_01X01, J19 CONN_01X01, J2 CONN_01X01, J20 Conn_02x04_Odd_Even, J21 CONN_01X01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

Commit message: artwork, aligning, checking, polishing..
Parts:
- C15: footprint Capacitor_THT:CP_Radial_D10.0mm_P5.00mm -> SNPM:CP_Radial_D10.0mm_P5.00mm_bottom
- LOGO1: footprint graphics:drawing -> graphics:PCB_artwork
- moved LOGO1 4.53 mm to (164.7, 89.9)
Other:
- board text added: "MAINBOARD 1.0"

Commit message: SENSORICNET mother board v.: 1.0
Parts:
- added C34: 47u, Capacitor_SMD:C_0805_2012Metric, F.Cu at (181.9, 118.4)
- C10, C11: value NC -> DNP
- C4, C6, C8, C9: value C -> 100n
- D10: value LED -> GREEN
- D2: value LED -> LED GREEN
- D8: value LED -> LED RED
- D9: value LED -> LED YELLOW
- J8: value Conn_01x02_Female -> Conn_02x01; footprint Connector_PinSocket_2.54mm:PinSocket_1x02_P2.54mm_Vertical -> Connector_PinHeader_2.54mm:PinHeader_1x02_P2.54mm_Vertical
- R1, R27, R28, R29: value R -> 1k
- R22: value 8k2 -> 1k6
- R23: value 5k6 -> 1k
- moved C17 7.68 mm to (184.4, 110.7), turned to 0 degrees
- moved C26 6.62 mm to (184.4, 112.8), turned to 0 degrees
- moved J7 2.54 mm to (173.3, 84.8)
- moved L4 2.33 mm to (183.3, 115.2), turned to 270 degrees
- moved D2 1.62 mm to (190.4, 55.0), turned to 0 degrees
- moved L7 1.57 mm to (187.9, 80.8)
- moved D11 1.46 mm to (155.7, 113.5)
- moved D1 1.46 mm to (188.0, 77.0)
- moved C27 1.41 mm to (185.1, 80.4)
- moved C28 1.40 mm to (183.8, 77.7)
- moved C25 1.38 mm to (185.8, 77.7)
- moved L5 0.74 mm to (135.8, 112.3)
- moved SW1 0.06 mm to (172.8, 124.3)
Connections:
- net reset renamed Net-(SW1-Pad2)
- U6 pad 2: (no net) -> Net-(C20-Pad1)
- U6 pad 7: (no net) -> Net-(R22-Pad2)
Routing:
- net GND: track 144.1 -> 171.5 mm, vias 53 -> 72
- net Net-(C17-Pad1): track 44.3 -> 37.3 mm, vias 3 -> 2
- net Net-(R22-Pad2): track 2.27 -> 7.30 mm
- net OLED_RESET: track 50.2 -> 52.8 mm
- net OLED_D/C: track 44.3 -> 46.9 mm
- net OLED_CS: track 39.9 -> 42.4 mm
- net Net-(D2-Pad2): track 22.6 -> 25.1 mm
- net USART_debug_rx: track 25.4 -> 27.5 mm
- net Net-(C30-Pad1): track 9.31 -> 11.4 mm
- net +5V: track 33.8 -> 31.8 mm, vias 2 -> 1
- net PM_SCK: track 24.6 -> 22.6 mm
- net gps_pulses: track 62.8 -> 60.9 mm
- net gps_reset: track 64.2 -> 62.3 mm
- net gps_standby: track 63.5 -> 61.7 mm
- net +3V3: track 214.0 -> 212.5 mm
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Other:
- net class Default: trace_width 0.5 -> 0.4
- board text added: "+5V"
- board text added: "+5V | +5V"
- board text added: "3V3"
- board text added: "AD 0"
- board text added: "AD 1"
- board text added: "CLK"
- board text added: "CLK | GND"
- board text added: "CS"
- board text added: "DBG TX | DBG RX"
- board text added: "DC"
- board text added: "DIO | RX"
- board text added: "GND"
- board text added: "GND | GND"
- board text added: "GND | GPS PULSES"
- board text added: "GND | TX"
- board text added: "GND_A"
- board text added: "GPS FIX"
- board text added: "GPS FIX | WIRELESS RESET"
- board text added: "GPS RESET | GPS STANDBY"
- board text added: "GPS TX | GPS RX"
- board text added: "RESET"
- board text added: "SCK"
- board text added: "SDA"
- board text added: "SDO"
- board text added: "[MODE]"
- board text added: "[RESET]"
- board text removed: "SW1"
- board text removed: "SW3"
- board text removed: "check pico clasp wiring"
- board text removed: "enable a led je prehozeny"

Commit message: priprava FAB data
Parts:
- D10: value GREEN -> LED GREEN
- moved C28 0.81 mm to (183.0, 77.7)
- moved C25 0.79 mm to (185.0, 77.7)
- moved D1 0.26 mm to (187.7, 77.0)
Other:
- net class Default: trace_width 0.4 -> 0.5
Changed lines of the file:
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@@
     (thickness 1.6)
     (drawings 92)
-    (tracks 1179)
+    (tracks 1181)
     (zones 0)
     (modules 98)
@@
   (layers
     (0 F.Cu signal)
-    (31 B.Cu signal)
+    (31 B.Cu signal hide)
     (32 B.Adhes user)
     (33 F.Adhes user)
@@
   )
   (setup
-    (last_trace_width 0.4)
+    (last_trace_width 0.5)
     (trace_clearance 0.15)
     (zone_clearance 0.2)
@@
       (drillshape 0)
       (scaleselection 1)
-      (outputdirectory "krivky/"))
+      (outputdirectory "FAB_outputs/machine/"))
   )
   (net 0 "")
@@
   (net_class Default "This is the default net class."
     (clearance 0.15)
-    (trace_width 0.4)
+    (trace_width 0.5)
     (via_dia 0.6)
     (via_drill 0.4)
@@
       (effects (font (size 1 1) (thickness 0.15)) (justify mirror))
     )
-    (fp_text value GREEN (at 0 1.75 180) (layer B.Fab)
+    (fp_text value "LED GREEN" (at 0 1.75 180) (layer B.Fab)
       (effects (font (size 1 1) (thickness 0.15)) (justify mirror))
     )
@@
   )
   (module Capacitor_SMD:C_0805_2012Metric (layer F.Cu)
-    (at 183.78932 77.68566 90)
+    (at 182.97652 77.68336 90)
     (descr "Capacitor SMD 0805 (2012 Metric), square (rectangular) end terminal, IPC_7351 nominal, (Body size source: https://docs.google.com/spreadsheets/d/1BsfQQcO9C6DZCsRaXUlFlo91Tg2WpOkGARC1WS5S8t0/edit?usp=sharing), generated with kicad-footprint-generator")
     (tags capacitor)
@@
   )
   (module Capacitor_SMD:C_0805_2012Metric (layer F.Cu)
-    (at 185.77052 77.68566 90)
+    (at 184.98312 77.68336 90)
     (descr "Capacitor SMD 0805 (2012 Metric), square (rectangular) end terminal, IPC_7351 nominal, (Body size source: https://docs.google.com/spreadsheets/d/1BsfQQcO9C6DZCsRaXUlFlo91Tg2WpOkGARC1WS5S8t0/edit?usp=sharing), generated with kicad-footprint-generator")
     (tags capacitor)
@@
   )
   (module Diode_SMD:D_SOD-123 (layer F.Cu)
-    (at 187.95492 76.99856 90)
+    (at 187.70092 76.97216 90)
     (descr SOD-123)
     (tags SOD-123)
@@
   (segment (start 191.05372 85.78216) (end 189.71452 87.12136) (width 0.5) (layer F.Cu) (net 3) (status 20))
   (segment (start 191.05372 85.43036) (end 191.05372 85.78216) (width 0.5) (layer F.Cu) (net 3))
-  (segment (start 183.78932 78.62316) (end 185.77052 78.62316) (width 0.5) (layer F.Cu) (net 3) (status 30))
   (segment (start 187.92952 78.62316) (end 187.95492 78.64856) (width 0.5) (layer F.Cu) (net 3) (status 30))
-  (segment (start 185.77052 78.62316) (end 187.92952 78.62316) (width 0.5) (layer F.Cu) (net 3) (status 30))
   (segment (start 187.58592 80.42656) (end 187.92952 80.08296) (width 0.5) (layer F.Cu) (net 3) (status 20))
   (segment (start 185.99682 80.42656) (end 187.58592 80.42656) (width 0.5) (layer F.Cu) (net 3) (status 10))
   (segment (start 187.92952 78.67396) (end 187.95492 78.64856) (width 0.5) (layer F.Cu) (net 3) (status 30))
-  (segment (start 187.92952 80.08296) (end 187.92952 78.67396) (width 0.5) (layer F.Cu) (net 3) (status 30))
-  (segment (start 182.57012 77.40396) (end 183.78932 78.62316) (width 0.5) (layer F.Cu) (net 3) (status 20))
-  (segment (start 179.42052 77.40396) (end 182.57012 77.40396) (width 0.5) (layer F.Cu) (net 3) (status 10))
   (segment (start 186.03722 80.46696) (end 185.99682 80.42656) (width 0.5) (layer F.Cu) (net 3) (status 30))
   (segment (start 186.03722 84.78266) (end 186.03722 80.46696) (width 0.5) (layer F.Cu) (net 3) (status 30))
@@
   (segment (start 187.92952 80.08296) (end 188.95752 80.08296) (width 0.5) (layer F.Cu) (net 3) (status 10))
   (segment (start 191.11722 82.24266) (end 193.65722 82.24266) (width 0.5) (layer B.Cu) (net 3) (status 30))
+  (segment (start 182.97652 78.62086) (end 184.98312 78.62086) (width 0.5) (layer F.Cu) (net 3) (status 30))
+  (segment (start 187.69962 78.62086) (end 187.70092 78.62216) (width 0.5) (layer F.Cu) (net 3) (status 30))
+  (segment (start 184.98312 78.62086) (end 187.69962 78.62086) (width 0.5) (layer F.Cu) (net 3) (status 30))
+  (segment (start 187.70092 79.85436) (end 187.92952 80.08296) (width 0.5) (layer F.Cu) (net 3) (status 30))
+  (segment (start 187.70092 78.62216) (end 187.70092 79.85436) (width 0.5) (layer F.Cu) (net 3) (status 30))
+  (segment (start 180.63742 78.62086) (end 179.42052 77.40396) (width 0.5) (layer F.Cu) (net 3) (status 20))
+  (segment (start 182.97652 78.62086) (end 180.63742 78.62086) (width 0.5) (layer F.Cu) (net 3) (status 10))
   (segment (start 191.1985 69.712754) (end 191.1985 69.469) (width 0.15) (layer F.Cu) (net 4) (status 30))
   (via (at 184.85612 68.08216) (size 0.6) (drill 0.4) (layers F.Cu B.Cu) (net 4))

Commit message: uklid
Parts:
- moved LOGO1 1.32 mm to (164.7, 91.2)
Other:
- board text added: "+5V|+5V"
- board text added: "CLK|GND"
- board text added: "DBG TX|DBG RX"
- board text added: "DIO|RX"
- board text added: "GND|GND"
- board text added: "GND|GPS PULSES"
- board text added: "GND|TX"
- board text added: "GPS FIX|WIRELESS RESET"
- board text added: "GPS RESET|GPS STANDBY"
- board text added: "GPS TX|GPS RX"
- board text removed: "+5V | +5V"
- board text removed: "CLK | GND"
- board text removed: "DBG TX | DBG RX"
- board text removed: "DIO | RX"
- board text removed: "GND | GND"
- board text removed: "GND | GPS PULSES"
- board text removed: "GND | TX"
- board text removed: "GPS FIX | WIRELESS RESET"
- board text removed: "GPS RESET | GPS STANDBY"
- board text removed: "GPS TX | GPS RX"
Changed lines of the file:
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@@
   (layers
     (0 F.Cu signal)
-    (31 B.Cu signal hide)
+    (31 B.Cu signal)
     (32 B.Adhes user)
     (33 F.Adhes user)
@@
     (aux_axis_origin 0 0)
     (grid_origin 174.67072 71.13016)
-    (visible_elements FFFFFFFF)
+    (visible_elements FFF9FFFF)
     (pcbplotparams
       (layerselection 0x01000_fffffffe)
@@
   )
   (module graphics:PCB_artwork (layer F.Cu)
-    (at 164.68852 89.87536)
+    (at 164.73932 91.19616)
     (fp_text reference LOGO1 (at 0 0) (layer F.SilkS) hide
       (effects (font (size 1.27 1.27) (thickness 0.15)))
@@
       (effects (font (size 1 1) (thickness 0.15)))
     )
-    (fp_line (start -3.81 -1.27) (end 0.27 -1.27) (layer F.Fab) (width 0.1))
-    (fp_line (start 0.27 -1.27) (end 1.27 -0.27) (layer F.Fab) (width 0.1))
-    (fp_line (start 1.27 -0.27) (end 1.27 8.89) (layer F.Fab) (width 0.1))
-    (fp_line (start 1.27 8.89) (end -3.81 8.89) (layer F.Fab) (width 0.1))
-    (fp_line (start -3.81 8.89) (end -3.81 -1.27) (layer F.Fab) (width 0.1))
-    (fp_line (start -3.87 -1.33) (end -1.27 -1.33) (layer F.SilkS) (width 0.12))
-    (fp_line (start -3.87 -1.33) (end -3.87 8.95) (layer F.SilkS) (width 0.12))
-    (fp_line (start -3.87 8.95) (end 1.33 8.95) (layer F.SilkS) (width 0.12))
-    (fp_line (start 1.33 1.27) (end 1.33 8.95) (layer F.SilkS) (width 0.12))
-    (fp_line (start -1.27 1.27) (end 1.33 1.27) (layer F.SilkS) (width 0.12))
-    (fp_line (start -1.27 -1.33) (end -1.27 1.27) (layer F.SilkS) (width 0.12))
-    (fp_line (start 1.33 -1.33) (end 1.33 0) (layer F.SilkS) (width 0.12))
-    (fp_line (start 0 -1.33) (end 1.33 -1.33) (layer F.SilkS) (width 0.12))
-    (fp_line (start -4.34 -1.8) (end 1.76 -1.8) (layer F.CrtYd) (width 0.05))
-    (fp_line (start 1.76 -1.8) (end 1.76 9.4) (layer F.CrtYd) (width 0.05))
-    (fp_line (start 1.76 9.4) (end -4.34 9.4) (layer F.CrtYd) (width 0.05))
-    (fp_line (start -4.34 9.4) (end -4.34 -1.8) (layer F.CrtYd) (width 0.05))
     (fp_text user %R (at -1.371001 3.889999 90) (layer F.Fab)
       (effects (font (size 1 1) (thickness 0.15)))
     )
-    (pad 1 thru_hole rect (at 0 0) (size 1.7 1.7) (drill 1) (layers *.Cu *.Mask)
-      (net 17 SWD_DIO))
-    (pad 2 thru_hole oval (at -2.54 0) (size 1.7 1.7) (drill 1) (layers *.Cu *.Mask)
-      (net 21 Rx))
-    (pad 3 thru_hole oval (at 0 2.54) (size 1.7 1.7) (drill 1) (layers *.Cu *.Mask)
-      (net 1 GND))
-    (pad 4 thru_hole oval (at -2.54 2.54) (size 1.7 1.7) (drill 1) (layers *.Cu *.Mask)
-      (net 22 Tx))
-    (pad 5 thru_hole oval (at 0 5.08) (size 1.7 1.7) (drill 1) (layers *.Cu *.Mask)
-      (net 16 SWD_CLK))
-    (pad 6 thru_hole oval (at -2.54 5.08) (size 1.7 1.7) (drill 1) (layers *.Cu *.Mask)
+    (fp_line (start -4.34 9.4) (end -4.34 -1.8) (layer F.CrtYd) (width 0.05))
+    (fp_line (start 1.76 9.4) (end -4.34 9.4) (layer F.CrtYd) (width 0.05))
+    (fp_line (start 1.76 -1.8) (end 1.76 9.4) (layer F.CrtYd) (width 0.05))
+    (fp_line (start -4.34 -1.8) (end 1.76 -1.8) (layer F.CrtYd) (width 0.05))
+    (fp_line (start 0 -1.33) (end 1.33 -1.33) (layer F.SilkS) (width 0.12))
+    (fp_line (start 1.33 -1.33) (end 1.33 0) (layer F.SilkS) (width 0.12))
+    (fp_line (start -1.27 -1.33) (end -1.27 1.27) (layer F.SilkS) (width 0.12))
+    (fp_line (start -1.27 1.27) (end 1.33 1.27) (layer F.SilkS) (width 0.12))
+    (fp_line (start 1.33 1.27) (end 1.33 8.95) (layer F.SilkS) (width 0.12))
+    (fp_line (start -3.87 8.95) (end 1.33 8.95) (layer F.SilkS) (width 0.12))
+    (fp_line (start -3.87 -1.33) (end -3.87 8.95) (layer F.SilkS) (width 0.12))
+    (fp_line (start -3.87 -1.33) (end -1.27 -1.33) (layer F.SilkS) (width 0.12))
+    (fp_line (start -3.81 8.89) (end -3.81 -1.27) (layer F.Fab) (width 0.1))
+    (fp_line (start 1.27 8.89) (end -3.81 8.89) (layer F.Fab) (width 0.1))
+    (fp_line (start 1.27 -0.27) (end 1.27 8.89) (layer F.Fab) (width 0.1))
+    (fp_line (start 0.27 -1.27) (end 1.27 -0.27) (layer F.Fab) (width 0.1))
+    (fp_line (start -3.81 -1.27) (end 0.27 -1.27) (layer F.Fab) (width 0.1))
+    (pad 8 thru_hole oval (at -2.54 7.62) (size 1.7 1.7) (drill 1) (layers *.Cu *.Mask)
       (net 1 GND))
     (pad 7 thru_hole oval (at 0 7.62) (size 1.7 1.7) (drill 1) (layers *.Cu *.Mask)
       (net 30 +3V3))
-    (pad 8 thru_hole oval (at -2.54 7.62) (size 1.7 1.7) (drill 1) (layers *.Cu *.Mask)
+    (pad 6 thru_hole oval (at -2.54 5.08) (size 1.7 1.7) (drill 1) (layers *.Cu *.Mask)
+      (net 1 GND))
+    (pad 5 thru_hole oval (at 0 5.08) (size 1.7 1.7) (drill 1) (layers *.Cu *.Mask)
+      (net 16 SWD_CLK))
+    (pad 4 thru_hole oval (at -2.54 2.54) (size 1.7 1.7) (drill 1) (layers *.Cu *.Mask)
+      (net 22 Tx))
+    (pad 3 thru_hole oval (at 0 2.54) (size 1.7 1.7) (drill 1) (layers *.Cu *.Mask)
       (net 1 GND))
+    (pad 2 thru_hole oval (at -2.54 0) (size 1.7 1.7) (drill 1) (layers *.Cu *.Mask)
+      (net 21 Rx))
+    (pad 1 thru_hole rect (at 0 0) (size 1.7 1.7) (drill 1) (layers *.Cu *.Mask)
+      (net 17 SWD_DIO))
     (model ${KISYS3DMOD}/Connector_PinSocket_2.54mm.3dshapes/PinSocket_2x04_P2.54mm_Vertical.wrl
       (at (xyz 0 0 0))
@@
     (effects (font (size 1 1) (thickness 0.25)) (justify mirror))
   )
-  (gr_text "CLK | GND" (at 139.23772 100.34016) (layer B.SilkS)
+  (gr_text CLK|GND (at 186.25312 102.65156) (layer B.SilkS)
     (effects (font (size 1 1) (thickness 0.25)) (justify mirror))
   )
-  (gr_text "DIO | RX" (at 139.61872 95.32366) (layer B.SilkS)
+  (gr_text DIO|RX (at 186.63412 97.63506) (layer B.SilkS)
     (effects (font (size 1 1) (thickness 0.25)) (justify mirror))
   )
-  (gr_text "GND | TX" (at 140.05052 97.91446) (layer B.SilkS)
+  (gr_text GND|TX (at 187.06592 100.22586) (layer B.SilkS)
     (effects (font (size 1 1) (thickness 0.25)) (justify mirror))
   )
@@
     (effects (font (size 1 1) (thickness 0.25)) (justify mirror))
   )
-  (gr_text +5V (at 186.93892 87.51316 90) (layer B.SilkS)
+  (gr_text +5V (at 186.10072 87.51316 90) (layer B.SilkS)
     (effects (font (size 1 1) (thickness 0.25)) (justify mirror))
   )
-  (gr_text SCK (at 185.36412 87.71636 90) (layer B.SilkS)
+  (gr_text SCK (at 183.53532 87.66556 90) (layer B.SilkS)
     (effects (font (size 1 1) (thickness 0.25)) (justify mirror))
   )
-  (gr_text SDO (at 183.68772 87.76716 90) (layer B.SilkS)
+  (gr_text SDO (at 180.99532 87.79256 90) (layer B.SilkS)
     (effects (font (size 1 1) (thickness 0.25)) (justify mirror))
   )
-  (gr_text DC (at 180.41112 87.23376 90) (layer B.SilkS)
+  (gr_text DC (at 175.81372 87.25916 90) (layer B.SilkS)
     (effects (font (size 1 1) (thickness 0.25)) (justify mirror))
   )
-  (gr_text RESET (at 182.06212 88.47836 90) (layer B.SilkS)
+  (gr_text RESET (at 178.53152 88.50376 90) (layer B.SilkS)
     (effects (font (size 1 1) (thickness 0.25)) (justify mirror))
   )
-  (gr_text CS (at 178.81092 87.20836 90) (layer B.SilkS)
+  (gr_text CS (at 173.14672 87.36076 90) (layer B.SilkS)
     (effects (font (size 1 1) (thickness 0.25)) (justify mirror))
   )
-  (gr_text "GND | GND" (at 147.44192 77.12456) (layer B.SilkS)
+  (gr_text GND|GND (at 147.41652 77.98816) (layer B.SilkS)
     (effects (font (size 1 1) (thickness 0.25)) (justify mirror))
   )
-  (gr_text "+5V | +5V" (at 147.44192 80.85836) (layer B.SilkS)
+  (gr_text +5V|+5V (at 147.36572 82.83956) (layer B.SilkS)
     (effects (font (size 1 1) (thickness 0.25)) (justify mirror))
   )
-  (gr_text "DBG TX | DBG RX" (at 147.34032 79.05496) (layer B.SilkS)
+  (gr_text "DBG TX|DBG RX" (at 147.26412 80.40116) (layer B.SilkS)
     (effects (font (size 1 1) (thickness 0.25)) (justify mirror))
   )
-  (gr_text "GPS FIX | WIRELESS RESET" (at 144.24152 75.29576) (layer B.SilkS)
+  (gr_text "GPS FIX|WIRELESS RESET" (at 144.24152 75.54976) (layer B.SilkS)
     (effects (font (size 1 1) (thickness 0.25)) (justify mirror))
   )
-  (gr_text "GPS RESET | GPS STANDBY" (at 146.47672 71.63816) (layer B.SilkS)
+  (gr_text "GPS RESET|GPS STANDBY" (at 146.50212 70.54596) (layer B.SilkS)
     (effects (font (size 1 1) (thickness 0.25)) (justify mirror))
   )
-  (gr_text "GND | GPS PULSES" (at 144.31772 69.83476) (layer B.SilkS)
+  (gr_text "GND|GPS PULSES" (at 144.31772 68.15836) (layer B.SilkS)
     (effects (font (size 1 1) (thickness 0.25)) (justify mirror))
   )
-  (gr_text "GND | GND" (at 147.49272 67.98056) (layer B.SilkS)
+  (gr_text GND|GND (at 147.46732 65.64376) (layer B.SilkS)
     (effects (font (size 1 1) (thickness 0.25)) (justify mirror))
   )
-  (gr_text "GPS TX | GPS RX" (at 147.36572 73.54316) (layer B.SilkS)
+  (gr_text "GPS TX|GPS RX" (at 147.36572 73.11136) (layer B.SilkS)
     (effects (font (size 1 1) (thickness 0.25)) (justify mirror))
   )

Commit message: pokracuju
Parts:
- removed SW3: SW_DPST, SNPM:edge_switch
- added C35: 1n, Capacitor_SMD:C_0805_2012Metric, F.Cu at (162.1, 94.9)
- added C36: 100n, Capacitor_SMD:C_0805_2012Metric, F.Cu at (173.8, 67.1)
- added D4: PTVS3V3S1UR,115, Diode_SMD:D_SOD-123, F.Cu at (185.6, 85.0)
- added J10: Conn_02x01, Connector_PinHeader_2.54mm:PinHeader_1x02_P2.54mm_Vertical, F.Cu at (163.0, 88.2)
- added J9: Conn_02x01, Connector_PinHeader_2.54mm:PinHeader_1x02_P2.54mm_Vertical, F.Cu at (163.0, 90.8)
- added LOGO2: LOGO, SNPM:OSHW-Logo2_9.8x8mm_BackSilkScreen, F.Cu at (142.6, 62.3)
- added SW2: SW_DPST, SNPM:edge_switch, F.Cu at (179.7, 124.2)
- C15: footprint SNPM:CP_Radial_D10.0mm_P5.00mm_bottom -> Capacitor_THT:CP_Radial_D10.0mm_P5.00mm
- J7: footprint Connector_PinHeader_2.54mm:PinHeader_1x07_P2.54mm_Vertical -> SNPM:OLED
- moved D2 83.1 mm to (145.9, 125.2)
- moved C15 51.2 mm to (145.8, 116.1), turned to 90 degrees
- moved D3 17.3 mm to (170.6, 121.0)
- moved C1 17.1 mm to (162.6, 109.9), turned to 0 degrees
- moved L3 16.2 mm to (164.1, 121.9)
- moved C2 14.2 mm to (162.6, 105.0), turned to 0 degrees
- moved L5 11.6 mm to (135.5, 100.7), turned to 0 degrees
- moved C20 10.6 mm to (140.6, 98.9), turned to 0 degrees
- moved D11 9.62 mm to (163.2, 107.5), turned to 0 degrees
- moved R13 9.28 mm to (166.7, 113.0), turned to 90 degrees
- moved J7 8.03 mm to (181.0, 82.2), turned to 0 degrees
- moved C18 7.61 mm to (153.7, 118.1)
- moved C22 7.35 mm to (140.6, 101.3), turned to 0 degrees
- moved U6 6.79 mm to (136.9, 107.8)
- moved R20 6.79 mm to (140.8, 107.1)
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Connections:
- J7 pad 1: OLED_CS -> GND
- J7 pad 2: OLED_D/C -> +5V
- J7 pad 3: OLED_RESET -> PM_SCK
- J7 pad 5: PM_SCK -> OLED_RESET
- J7 pad 6: +5V -> OLED_D/C
- J7 pad 7: GND -> OLED_CS
- R8 pad 1: Rx -> Net-(J10-Pad2)
- R9 pad 1: Tx -> Net-(J9-Pad2)
Routing:
- net Net-(D2-Pad2): track 25.1 -> 124.1 mm, vias 1 -> 3
- net +5V: track 31.7 -> 120.2 mm, vias 1 -> 3
- net GND: track 171.5 -> 215.4 mm, vias 72 -> 89
- net 5V_enable: track 40.3 -> 21.3 mm
- net +6V: track 43.7 -> 61.7 mm
- net Net-(D3-Pad2): track 33.6 -> 16.6 mm
- net OLED_RESET: track 52.8 -> 38.7 mm, vias 3 -> 1
- net Net-(SW2-Pad1): track 23.6 -> 32.4 mm
- net +3V3: track 212.5 -> 220.4 mm, vias 7 -> 9
- net Net-(R22-Pad2): track 7.30 -> 14.5 mm
- net Net-(C16-Pad1): track 10.6 -> 17.7 mm
- net Net-(J9-Pad2): track 0.00 -> 6.76 mm
- net Net-(J10-Pad2): track 0.00 -> 6.39 mm
- net Tx: track 46.3 -> 40.0 mm, vias 2 -> 1
- net OLED_D/C: track 46.9 -> 40.7 mm, vias 3 -> 1
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Other:
- net class Default: trace_width 0.5 -> 0.15
- board text added: "5V|5V"
- board text added: "GPS FIX|WIRELESS RES"
- board text added: "GPS RES|GPS STANDBY"
- board text removed: "+5V|+5V"
- board text removed: "DBG TX|DBG RX"
- board text removed: "GPS FIX|WIRELESS RESET"
- board text removed: "GPS RESET|GPS STANDBY"

Commit message: shield template added
Parts:
- added J12: Barrel_Jack_Switch, Connector_BarrelJack:BarrelJack_Horizontal, F.Cu at (188.2, 112.3)
- added J14: Conn_01x02_Female, Connector_PinHeader_2.54mm:PinHeader_1x02_P2.54mm_Vertical, F.Cu at (191.0, 121.6)
- J13: footprint Connector_Wire:SolderWirePad_1x02_P3.81mm_Drill1.2mm -> Connector_PinHeader_2.54mm:PinHeader_1x02_P2.54mm_Vertical
- moved J13 6.51 mm to (185.5, 121.6), turned to 0 degrees
- moved LOGO2 5.38 mm to (142.6, 67.7)
- moved C17 3.89 mm to (180.5, 110.7), turned to 180 degrees
- moved C26 3.86 mm to (180.5, 112.8), turned to 180 degrees
- moved LOGO1 2.25 mm to (163.3, 89.5)
- moved L4 1.96 mm to (181.4, 115.2)
Connections:
- D3 pad 2: Net-(D3-Pad2) -> +9V
- J13 pad 1: GND -> +9V
- J13 pad 2: Net-(D3-Pad2) -> +9V
Routing:
- net +9V: track 0.00 -> 27.7 mm
- net Net-(D3-Pad2): track 16.6 -> 0.00 mm
- net GND: track 215.4 -> 202.7 mm, vias 89 -> 86
- net Net-(D2-Pad2): track 124.1 -> 132.2 mm
- net +3V3: track 220.4 -> 224.3 mm, vias 9 -> 8
- net i2c_scl: track 19.2 -> 16.2 mm
- net i2c_sda: track 16.9 -> 15.5 mm
- net Net-(D10-Pad2): track 26.7 -> 25.5 mm
Other:
- net class Default: trace_width 0.15 -> 0.5
- board text added: "+"
- board text added: "SENSORICNET.COM"
- board text added: "VIN"
