File: hardware/NBIOT_mainboard/sensenet_particlemeter.sch (KiCad schematic (older format))
At the start: 97 parts, among them J1 CONN_01X01, J11 CONN_01X01, J13 Conn_01x02_Female, J16 Conn_01x06_Female, J17 Conn_02x08_Odd_Even, J18 CONN_01X01, J19 CONN_01X01, J2 CONN_01X01, J20 Conn_02x04_Odd_Even, J21 CONN_01X01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

Commit message: artwork, aligning, checking, polishing..
Parts:
- C15: footprint Capacitor_THT:CP_Radial_D10.0mm_P5.00mm -> SNPM:CP_Radial_D10.0mm_P5.00mm_bottom
- LOGO1: footprint graphics:drawing -> graphics:PCB_artwork
Changed lines of the file:
@@
 F 0 "C15" H 21075 1900 50  0000 L CNN
 F 1 "470u" H 21075 1700 50  0000 L CNN
-F 2 "Capacitor_THT:CP_Radial_D10.0mm_P5.00mm" H 21088 1650 50  0001 C CNN
+F 2 "SNPM:CP_Radial_D10.0mm_P5.00mm_bottom" H 21088 1650 50  0001 C CNN
 F 3 "" H 21050 1800 50  0001 C CNN
 	1    21050 1800
@@
 F 0 "LOGO1" H 21850 14350 60  0000 C CNN
 F 1 "LOGO" H 21850 13950 60  0000 C CNN
-F 2 "graphics:drawing" H 21850 14150 60  0001 C CNN
+F 2 "graphics:PCB_artwork" H 21850 14150 60  0001 C CNN
 F 3 "" H 21850 14150 60  0001 C CNN
 	1    21850 14150

Commit message: SENSORICNET mother board v.: 1.0
Parts:
- removed J8: Conn_01x02_Female, Connector_PinSocket_2.54mm:PinSocket_1x02_P2.54mm_Vertical, symbol Connector:Conn_01x02_Female
- added C34: 47u, Capacitor_SMD:C_0805_2012Metric, symbol sensenet_particlemeter-rescue:C
- added J8: Conn_02x01, Connector_PinHeader_2.54mm:PinHeader_1x02_P2.54mm_Vertical, symbol Connector_Generic:Conn_02x01
- C10, C11: value NC -> DNP
- C4, C6, C8, C9: value C -> 100n
- D10, D2: value LED -> LED GREEN
- D8: value LED -> LED RED
- D9: value LED -> LED YELLOW
- R1, R27, R28, R29: value R -> 1k
- R22: value 8k2 -> 1k6
- R23: value 5k6 -> 1k
Connections:
- net GND: now also C34.2
- net i2c_scl: now also J8.2 (Pin_2)
- net i2c_sda: now also J8.1 (Pin_1)
- net at C30.1, L4.2, R12.1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: now also C34.1
- net at R22.2, R23.1: now also U6.7 (ADJ)
- net at C20.1, C22.1, C3.1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: now also U6.2 (EN)
- net BOOT_0: no longer names the net of U2.60 (boot0)
- net BOOT_signal: no longer names the net of U2.61 (pb8)
- net debug_on_off: no longer names the net of U2.62 (pb9)
- net reset: no longer names the net of SW1.2, U2.7 (nrst)
- no-connect marks 80 -> 85
Other:
- note added: "ARTWORK"
- note added: "Connecting wire MOLEX s.n. 15133-0600 [50mm]"
- note added: "Connecting wire MOLEX s.n. 15133-0601 [100mm]"
- note added: "Connector MOLEX s.n. 501568-0607 [pico-clasp 6pos]"
- note added: "ESE477M025AH1EA kondenzator?"
- note added: "JTAG, I2C for external bme280"
- note added: "Molex pico clasp connector:"
- note added: "Mounting holes"
- note added: "OLED connector for 128x64, driver ssd1306, 7pin"
- note added: "Secure element"
- note added: "Shield connector, debug signals"
- note removed: "15133-0601"
- note removed: "501568-0607"
- note removed: "ESE477M025AH1EA"
- note removed: "pico clasp konektor,\n"
- note removed: "zamek ke mne, drat doprava, jednicla dole.\n6 gnd\n5 SS\n4 SDI\n3 SDO\n2 SCK\n1 VCC\n"
- moved on the sheet: C1, C10, C11, C12, C13, C14, C15, C16, C17, C18, C19, C2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

Commit message: pokracuju
Parts:
- added C35: 1n, Capacitor_SMD:C_0805_2012Metric, symbol sensenet_particlemeter-rescue:C
- added C36: 100n, Capacitor_SMD:C_0805_2012Metric, symbol sensenet_particlemeter-rescue:C
- added D4: PTVS3V3S1UR,115, Diode_SMD:D_SOD-123, symbol sensenet_particlemeter-rescue:D_Schottky
- added J10, J9: Conn_02x01, Connector_PinHeader_2.54mm:PinHeader_1x02_P2.54mm_Vertical, symbol Connector_Generic:Conn_02x01
- added LOGO2: LOGO, SNPM:OSHW-Logo2_9.8x8mm_BackSilkScreen, symbol sensenet_particlemeter-rescue:LOGO
- C15: footprint SNPM:CP_Radial_D10.0mm_P5.00mm_bottom -> Capacitor_THT:CP_Radial_D10.0mm_P5.00mm
- J7: footprint Connector_PinHeader_2.54mm:PinHeader_1x07_P2.54mm_Vertical -> SNPM:OLED
- renumbered SW3 to SW2
Connections:
- net +3V3: now also C35.1, C36.1
- net +5V: now also J7.2 (Pin_2); no longer J7.6 (Pin_6)
- net GND: now also J7.1 (Pin_1), C35.2, C36.2, D4.2 (A); no longer J7.7 (Pin_7)
- net OLED_CS: now also J7.7 (Pin_7); no longer J7.1 (Pin_1)
- net OLED_D/C: now also J7.6 (Pin_6); no longer J7.2 (Pin_2)
- net OLED_RESET: now also J7.5 (Pin_5); no longer J7.3 (Pin_3)
- net PM_SCK: now also J7.3 (Pin_3); no longer J7.5 (Pin_5)
- net Rx: now also J10.1 (Pin_1); no longer R8.1
- net Tx: now also J9.1 (Pin_1); no longer R9.1
- net at C17.1, C26.1, L4.1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: now also D4.1 (K)
- new net: J10.2 (Pin_2), R8.1
- new net: J9.2 (Pin_2), R9.1
Other:
- note added: "OPEN HARDWARE"
- moved on the sheet: C14, C17, C26, L7, LOGO1
Changed lines of the file:
@@
 	1    0    0    -1
 $EndComp
-Text GLabel 2850 14400 0    39   Input ~ 0
+Text GLabel 2250 14400 0    39   Input ~ 0
 Rx
-Text GLabel 2800 13650 0    39   Input ~ 0
+Text GLabel 2200 13650 0    39   Input ~ 0
 Tx
 $Comp
@@
 L sensenet_particlemeter-rescue:C C14
 U 1 1 59A56B77
-P 9450 4200
-F 0 "C14" H 9475 4300 50  0000 L CNN
-F 1 "2,2u" H 9475 4100 50  0000 L CNN
-F 2 "Capacitor_SMD:C_0805_2012Metric" H 9488 4050 50  0001 C CNN
-F 3 "" H 9450 4200 50  0001 C CNN
-	1    9450 4200
+P 9450 4250
+F 0 "C14" H 9475 4350 50  0000 L CNN
+F 1 "2,2u" H 9475 4150 50  0000 L CNN
+F 2 "Capacitor_SMD:C_0805_2012Metric" H 9488 4100 50  0001 C CNN
+F 3 "" H 9450 4250 50  0001 C CNN
+	1    9450 4250
 	1    0    0    -1
 $EndComp
@@
 L sensenet_particlemeter-rescue:GND #PWR034
 U 1 1 59A5DDD4
-P 9450 4450
-F 0 "#PWR034" H 9450 4200 50  0001 C CNN
-F 1 "GND" H 9450 4300 50  0000 C CNN
-F 2 "" H 9450 4450 50  0001 C CNN
-F 3 "" H 9450 4450 50  0001 C CNN
-	1    9450 4450
+P 9450 5400
+F 0 "#PWR034" H 9450 5150 50  0001 C CNN
+F 1 "GND" H 9450 5250 50  0000 C CNN
+F 2 "" H 9450 5400 50  0001 C CNN
+F 3 "" H 9450 5400 50  0001 C CNN
+	1    9450 5400
 	1    0    0    -1
 $EndComp
@@
 F 0 "C15" H 20825 2500 50  0000 L CNN
 F 1 "470u" H 20825 2300 50  0000 L CNN
-F 2 "SNPM:CP_Radial_D10.0mm_P5.00mm_bottom" H 20838 2250 50  0001 C CNN
+F 2 "Capacitor_THT:CP_Radial_D10.0mm_P5.00mm" H 20838 2250 50  0001 C CNN
 F 3 "" H 20800 2400 50  0001 C CNN
 	1    20800 2400
@@
 $EndComp
 $Comp
-L sensenet_particlemeter-rescue:SW_DPST SW3
+L sensenet_particlemeter-rescue:SW_DPST SW2
 U 1 1 5B501DB8
 P 5650 7500
-F 0 "SW3" H 5650 7700 50  0000 C CNN
+F 0 "SW2" H 5650 7700 50  0000 C CNN
 F 1 "SW_DPST" H 5650 7300 50  0000 C CNN
 F 2 "SNPM:edge_switch" H 5650 7500 50  0001 C CNN
@@
 L sensenet_particlemeter-rescue:Ferrite_Bead L7
 U 1 1 5BA78A59
-P 20550 2150
-F 0 "L7" V 20400 2175 50  0000 C CNN
-F 1 "FBMH1608HL601-T" V 20250 2300 50  0000 C CNN
-F 2 "Resistors_SMD:R_0603" V 20480 2150 50  0001 C CNN
-F 3 "" H 20550 2150 50  0000 C CNN
-	1    20550 2150
+P 20650 2150
+F 0 "L7" V 20500 2175 50  0000 C CNN
+F 1 "FBMH1608HL601-T" V 20350 2300 50  0000 C CNN
+F 2 "Resistors_SMD:R_0603" V 20580 2150 50  0001 C CNN
+F 3 "" H 20650 2150 50  0000 C CNN
+	1    20650 2150
 	0    1    1    0
 $EndComp
@@
 	0    -1   1    0
 $EndComp
-Wire Wire Line
-	20700 2150 20800 2150
 Connection ~ 20800 2150
 Wire Wire Line
@@
 	9800 3900 10050 3900
 Wire Wire Line
-	8900 4050 9450 4050
-Connection ~ 9450 4050
-Wire Wire Line
-	9450 4350 9450 4450
-Wire Wire Line
 	11450 4200 12600 4200
 Wire Wire Line
@@
 L sensenet_particlemeter-rescue:LOGO LOGO1
 U 1 1 5BA9EC4C
-P 11050 13750
-F 0 "LOGO1" H 11050 13950 60  0000 C CNN
-F 1 "LOGO" H 11050 13550 60  0000 C CNN
-F 2 "graphics:PCB_artwork" H 11050 13750 60  0001 C CNN
-F 3 "" H 11050 13750 60  0001 C CNN
-	1    11050 13750
+P 8850 13750
+F 0 "LOGO1" H 8850 13950 60  0000 C CNN
+F 1 "LOGO" H 8850 13550 60  0000 C CNN
+F 2 "graphics:PCB_artwork" H 8850 13750 60  0001 C CNN
+F 3 "" H 8850 13750 60  0001 C CNN
+	1    8850 13750
 	1    0    0    -1
 $EndComp
@@
 	10550 3250 10700 3250
 Wire Wire Line
-	9450 4050 9800 4050
-Wire Wire Line
 	6150 10050 6150 10100
 Wire Wire Line
@@
 L sensenet_particlemeter-rescue:C C17
 U 1 1 5C619B52
-P 20050 2400
-F 0 "C17" H 20075 2500 50  0000 L CNN
-F 1 "100n" H 20075 2300 50  0000 L CNN
-F 2 "Capacitor_SMD:C_0805_2012Metric" H 20088 2250 50  0001 C CNN
-F 3 "" H 20050 2400 50  0001 C CNN
-	1    20050 2400
+P 20250 2400
+F 0 "C17" H 20275 2500 50  0000 L CNN
+F 1 "100n" H 20275 2300 50  0000 L CNN
+F 2 "Capacitor_SMD:C_0805_2012Metric" H 20288 2250 50  0001 C CNN
+F 3 "" H 20250 2400 50  0001 C CNN
+	1    20250 2400
 	1    0    0    -1
 $EndComp
@@
 L sensenet_particlemeter-rescue:C C26
 U 1 1 5C721A42
-P 20300 2400
-F 0 "C26" H 20325 2500 50  0000 L CNN
-F 1 "1n" H 20325 2300 50  0000 L CNN
-F 2 "Capacitor_SMD:C_0805_2012Metric" H 20338 2250 50  0001 C CNN
-F 3 "" H 20300 2400 50  0001 C CNN
-	1    20300 2400
+P 20450 2400
+F 0 "C26" H 20475 2500 50  0000 L CNN
+F 1 "1n" H 20475 2300 50  0000 L CNN
+F 2 "Capacitor_SMD:C_0805_2012Metric" H 20488 2250 50  0001 C CNN
+F 3 "" H 20450 2400 50  0001 C CNN
+	1    20450 2400
 	1    0    0    -1
 $EndComp
@@
 $EndComp
 Wire Wire Line
-	20050 2250 20050 2150
-Connection ~ 20050 2150
+	20250 2250 20250 2150
+Connection ~ 20250 2150
 Wire Wire Line
-	20050 2150 20300 2150
+	20250 2150 20450 2150
 Wire Wire Line
-	20300 2250 20300 2150
-Connection ~ 20300 2150
+	20450 2250 20450 2150
+Connection ~ 20450 2150
 Wire Wire Line
-	20050 2550 20050 3050
+	20250 2550 20250 3050
 Wire Wire Line
-	20050 3050 20300 3050
+	20250 3050 20450 3050
 Wire Wire Line
-	20300 2550 20300 3050
-Connection ~ 20300 3050
+	20450 2550 20450 3050
+Connection ~ 20450 3050
 $Comp
 L sensenet_particlemeter-rescue:C C27
@@
 $EndComp
 Wire Wire Line
-	20300 2150 20400 2150
+	20450 2150 20500 2150
 Wire Wire Line
-	20300 3050 20600 3050
+	20450 3050 20600 3050
 Wire Wire Line
 	21350 2550 21350 3050
@@
 F 0 "J7" H 20927 11026 50  0000 L CNN
 F 1 "Conn_01x07_Female" H 20927 10935 50  0000 L CNN
-F 2 "Connector_PinHeader_2.54mm:PinHeader_1x07_P2.54mm_Vertical" H 20900 11000 50  0001 C CNN
+F 2 "SNPM:OLED" H 20900 11000 50  0001 C CNN
 F 3 "~" H 20900 11000 50  0001 C CNN
 	1    20900 11000
-	1    0    0    -1
+	1    0    0    1
 $EndComp
 Wire Wire Line
@@
 	8300 9750 8300 12350
 Connection ~ 10050 4350
+$Comp
+L sensenet_particlemeter-rescue:D_Schottky D4
+U 1 1 5C8856DB
+P 20050 2650
+F 0 "D4" H 20050 2750 50  0000 C CNN
+F 1 "PTVS3V3S1UR,115" H 20050 2550 50  0000 C CNN
+F 2 "Diode_SMD:D_SOD-123" H 20050 2650 50  0001 C CNN
+F 3 "" H 20050 2650 50  0001 C CNN
+	1    20050 2650
+	0    1    1    0
+$EndComp
+$Comp
+L sensenet_particlemeter-rescue:GND #PWR0128
+U 1 1 5C8857ED
+P 20050 3550
+F 0 "#PWR0128" H 20050 3300 50  0001 C CNN
+F 1 "GND" H 20050 3400 50  0000 C CNN
+F 2 "" H 20050 3550 50  0001 C CNN
+F 3 "" H 20050 3550 50  0001 C CNN
+	1    20050 3550
+	1    0    0    -1
+$EndComp
+Wire Wire Line
+	20050 2500 20050 2150
+Connection ~ 20050 2150
+Wire Wire Line
+	20050 2150 20250 2150
+Wire Wire Line
+	20050 2800 20050 3550
+$Comp
+L Connector_Generic:Conn_02x01 J9
+U 1 1 5C8E8AA3
+P 2500 13650
+F 0 "J9" H 2550 13867 50  0000 C CNN
+F 1 "Conn_02x01" H 2550 13776 50  0000 C CNN
+F 2 "Connector_PinHeader_2.54mm:PinHeader_1x02_P2.54mm_Vertical" H 2500 13650 50  0001 C CNN
+F 3 "~" H 2500 13650 50  0001 C CNN
+	1    2500 13650
+	1    0    0    -1
+$EndComp
+$Comp
+L Connector_Generic:Conn_02x01 J10
+U 1 1 5C8E9383
+P 2550 14400
+F 0 "J10" H 2600 14617 50  0000 C CNN
+F 1 "Conn_02x01" H 2600 14526 50  0000 C CNN
+F 2 "Connector_PinHeader_2.54mm:PinHeader_1x02_P2.54mm_Vertical" H 2550 14400 50  0001 C CNN
+F 3 "~" H 2550 14400 50  0001 C CNN
+	1    2550 14400
+	1    0    0    -1
+$EndComp
+Wire Wire Line
+	2200 13650 2300 13650
+Wire Wire Line
+	2250 14400 2350 14400
+$Comp
+L sensenet_particlemeter-rescue:LOGO LOGO2
+U 1 1 5C9B9E15
+P 10350 13750
+F 0 "LOGO2" H 10350 13950 60  0000 C CNN
+F 1 "LOGO" H 10350 13550 60  0000 C CNN
+F 2 "SNPM:OSHW-Logo2_9.8x8mm_BackSilkScreen" H 10350 13750 60  0001 C CNN
+F 3 "" H 10350 13750 60  0001 C CNN
+	1    10350 13750
+	1    0    0    -1
+$EndComp
+Text Notes 10000 12750 0    60   ~ 0
+OPEN HARDWARE
+$Comp
+L sensenet_particlemeter-rescue:C C35
+U 1 1 5C9BBF2F
+P 1400 5050
+F 0 "C35" H 1425 5150 50  0000 L CNN
+F 1 "1n" H 1425 4950 50  0000 L CNN
+F 2 "Capacitor_SMD:C_0805_2012Metric" H 1438 4900 50  0001 C CNN
+F 3 "" H 1400 5050 50  0001 C CNN
+	1    1400 5050
+	1    0    0    -1
+$EndComp
+Wire Wire Line
+	1400 4900 1400 4850
+Wire Wire Line
+	1400 4850 1800 4850
+Wire Wire Line
+	1400 5200 1400 5250
+Wire Wire Line
+	1400 5250 1800 5250
+Connection ~ 1800 5250
+$Comp
+L sensenet_particlemeter-rescue:C C36
+U 1 1 5CA22E9E
+P 9150 4250
+F 0 "C36" H 9175 4350 50  0000 L CNN
+F 1 "100n" H 9175 4150 50  0000 L CNN
+F 2 "Capacitor_SMD:C_0805_2012Metric" H 9188 4100 50  0001 C CNN
+F 3 "" H 9150 4250 50  0001 C CNN
+	1    9150 4250
+	1    0    0    -1
+$EndComp
+Wire Wire Line
+	9450 5400 9450 4400
+Wire Wire Line
+	8900 4050 9150 4050
+Wire Wire Line
+	9150 4100 9150 4050
+Connection ~ 9150 4050
+Wire Wire Line
+	9150 4050 9450 4050
+Wire Wire Line
+	9450 4100 9450 4050
+Connection ~ 9450 4050
+Wire Wire Line
+	9450 4050 9800 4050
+$Comp
+L sensenet_particlemeter-rescue:GND #PWR0129
+U 1 1 5CB243A6
+P 9150 5400
+F 0 "#PWR0129" H 9150 5150 50  0001 C CNN
+F 1 "GND" H 9150 5250 50  0000 C CNN
+F 2 "" H 9150 5400 50  0001 C CNN
+F 3 "" H 9150 5400 50  0001 C CNN
+	1    9150 5400
+	1    0    0    -1
+$EndComp
+Wire Wire Line
+	9150 4400 9150 5400
 $EndSCHEMATC

Commit message: shield template added
Parts:
- added J12: Barrel_Jack_Switch, Connector_BarrelJack:BarrelJack_Horizontal, symbol Connector:Barrel_Jack_Switch
- added J14: Conn_01x02_Female, Connector_PinHeader_2.54mm:PinHeader_1x02_P2.54mm_Vertical, symbol Connector:Conn_01x02_Female
- J13: footprint Connector_Wire:SolderWirePad_1x02_P3.81mm_Drill1.2mm -> Connector_PinHeader_2.54mm:PinHeader_1x02_P2.54mm_Vertical
Connections:
- net labels added: +9V
- wire segments 450 -> 463
Other:
- moved on the sheet: J13
Changed lines of the file:
@@
 P 15050 2150
 F 0 "D3" H 15050 2250 50  0000 C CNN
-F 1 "D_Schottky_ss14" H 15100 2000 50  0000 C CNN
+F 1 "D_Schottky_ss14" V 15050 1700 50  0000 C CNN
 F 2 "Diode_SMD:D_SOD-123" H 15050 2150 50  0001 C CNN
 F 3 "" H 15050 2150 50  0001 C CNN
@@
 	15600 2050 15600 2150
 Wire Wire Line
-	14850 2150 14900 2150
-Wire Wire Line
 	15550 2150 15600 2150
 Wire Wire Line
@@
 L Connector:Conn_01x02_Female J13
 U 1 1 5C6AC441
-P 14650 2250
-F 0 "J13" H 14544 1925 50  0000 C CNN
-F 1 "Conn_01x02_Female" V 14750 2350 50  0000 C CNN
-F 2 "Connector_Wire:SolderWirePad_1x02_P3.81mm_Drill1.2mm" H 14650 2250 50  0001 C CNN
-F 3 "~" H 14650 2250 50  0001 C CNN
-	1    14650 2250
+P 14550 2150
+F 0 "J13" H 14500 2250 50  0000 C CNN
+F 1 "Conn_01x02_Female" V 14650 1750 50  0000 C CNN
+F 2 "Connector_PinHeader_2.54mm:PinHeader_1x02_P2.54mm_Vertical" H 14550 2150 50  0001 C CNN
+F 3 "~" H 14550 2150 50  0001 C CNN
+	1    14550 2150
 	-1   0    0    1
 $EndComp
-Wire Wire Line
-	14850 2250 14850 3550
 $Comp
 L NCP59152:NCP59152 U1
@@
 P 15600 2050
 F 0 "#PWR0106" H 15600 1900 50  0001 C CNN
-F 1 "+6V" H 15615 2223 50  0000 C CNN
+F 1 "+6V" H 15600 2200 50  0000 C CNN
 F 2 "" H 15600 2050 50  0001 C CNN
 F 3 "" H 15600 2050 50  0001 C CNN
@@
 Wire Wire Line
 	9150 4400 9150 5400
+$Comp
+L Connector:Barrel_Jack_Switch J12
+U 1 1 5C770C91
+P 14850 13300
+F 0 "J12" H 14905 13617 50  0000 C CNN
+F 1 "Barrel_Jack_Switch" H 14905 13526 50  0000 C CNN
+F 2 "Connector_BarrelJack:BarrelJack_Horizontal" H 14900 13260 50  0001 C CNN
+F 3 "~" H 14900 13260 50  0001 C CNN
+	1    14850 13300
+	1    0    0    -1
+$EndComp
+$Comp
+L power:+9V #PWR0130
+U 1 1 5C771EA1
+P 14900 2050
+F 0 "#PWR0130" H 14900 1900 50  0001 C CNN
+F 1 "+9V" H 14850 2200 50  0000 C CNN
+F 2 "" H 14900 2050 50  0001 C CNN
+F 3 "" H 14900 2050 50  0001 C CNN
+	1    14900 2050
+	1    0    0    -1
+$EndComp
+Wire Wire Line
+	14900 2050 14900 2150
+Connection ~ 14900 2150
+$Comp
+L power:+9V #PWR0131
+U 1 1 5C7A8760
+P 15400 13150
+F 0 "#PWR0131" H 15400 13000 50  0001 C CNN
+F 1 "+9V" H 15350 13300 50  0000 C CNN
+F 2 "" H 15400 13150 50  0001 C CNN
+F 3 "" H 15400 13150 50  0001 C CNN
+	1    15400 13150
+	1    0    0    -1
+$EndComp
+$Comp
+L sensenet_particlemeter-rescue:GND #PWR0132
+U 1 1 5C7A983C
+P 15400 13700
+F 0 "#PWR0132" H 15400 13450 50  0001 C CNN
+F 1 "GND" H 15400 13550 50  0000 C CNN
+F 2 "" H 15400 13700 50  0001 C CNN
+F 3 "" H 15400 13700 50  0001 C CNN
+	1    15400 13700
+	1    0    0    -1
+$EndComp
+Wire Wire Line
+	15150 13200 15400 13200
+Wire Wire Line
+	15400 13200 15400 13150
+Wire Wire Line
+	15150 13300 15400 13300
+Wire Wire Line
+	15400 13300 15400 13400
+Wire Wire Line
+	15150 13400 15400 13400
+Connection ~ 15400 13400
+Wire Wire Line
+	15400 13400 15400 13700
+$Comp
+L Connector:Conn_01x02_Female J14
+U 1 1 5C84CC5B
+P 14550 2550
+F 0 "J14" H 14500 2650 50  0000 C CNN
+F 1 "Conn_01x02_Female" V 14600 2850 50  0000 C CNN
+F 2 "Connector_PinHeader_2.54mm:PinHeader_1x02_P2.54mm_Vertical" H 14550 2550 50  0001 C CNN
+F 3 "~" H 14550 2550 50  0001 C CNN
+	1    14550 2550
+	-1   0    0    1
+$EndComp
+Wire Wire Line
+	14750 2050 14800 2050
+Wire Wire Line
+	14800 2050 14800 2150
+Wire Wire Line
+	14800 2150 14900 2150
+Wire Wire Line
+	14750 2150 14800 2150
+Connection ~ 14800 2150
+Wire Wire Line
+	14750 2450 14850 2450
+Wire Wire Line
+	14850 2450 14850 2550
+Wire Wire Line
+	14750 2550 14850 2550
+Connection ~ 14850 2550
+Wire Wire Line
+	14850 2550 14850 3550
 $EndSCHEMATC
